Commit message: fixed bug: gazebo control were not working. TODO: fix differential controller

File: urdf/m2wr_arm.xacro (robot description, xacro)
@@ -301,3 +301,43 @@
   	<child link="left_grip_link"/>
   </joint>
+<transmission name="arm_joint_01_trans">
+<type>transmission_interface/SimpleTransmission</type>
+<joint name="arm_joint_01">
+<hardwareInterface>hardware_interface/EffortJointInterface</hardwareInterface>
+</joint>
+<actuator name="motor1">
+<hardwareInterface>hardware_interface/EffortJointInterface</hardwareInterface>
+<mechanicalInterface>1</mechanicalInterface>
+</actuator>
+</transmission>
+<transmission name="arm_joint_02_trans">
+<type>transmission_interface/SimpleTransmission</type>
+<joint name="arm_joint_02">
+<hardwareInterface>hardware_interface/EffortJointInterface</hardwareInterface>
+</joint>
+<actuator name="motor2">
+<hardwareInterface>hardware_interface/EffortJointInterface</hardwareInterface>
+<mechanicalInterface>1</mechanicalInterface>
+</actuator>
+</transmission>
+<transmission name="arm_joint_03_trans">
+<type>transmission_interface/SimpleTransmission</type>
+<joint name="arm_joint_03">
+<hardwareInterface>hardware_interface/EffortJointInterface</hardwareInterface>
+</joint>
+<actuator name="motor3">
+<hardwareInterface>hardware_interface/EffortJointInterface</hardwareInterface>
+<mechanicalInterface>1</mechanicalInterface>
+</actuator>
+</transmission>
+<transmission name="arm_joint_04_trans">
+<type>transmission_interface/SimpleTransmission</type>
+<joint name="arm_joint_04">
+<hardwareInterface>hardware_interface/EffortJointInterface</hardwareInterface>
+</joint>
+<actuator name="motor4">
+<hardwareInterface>hardware_interface/EffortJointInterface</hardwareInterface>
+<mechanicalInterface>1</mechanicalInterface>
+</actuator>
+</transmission>
 </robot>

Commit message: robot shakes but it exists. In order to understand if it works well i need to fix this bug. Then i have to adjust the robot model in order to be a little bigger then I need to evaluate the fact that the robot is capable of moving (it is a mobile robots) then moveit, rosplan etc etc

File: urdf/m2wr_arm.xacro (robot description, xacro)
@@ -247,5 +247,5 @@
   	<child link="arm_link_04"/>
   </joint>
-<link name="right_grip_link">
+<link name="grip_link">
   	<inertial>
   		<mass value="0.01"/>
@@ -267,37 +267,10 @@
   	</visual>
   </link>
-  <joint name="right_grip_joint" type="prismatic">
+  <joint name="grip_joint" type="prismatic">
   	<axis xyz="1 0 0"/>
   	<limit effort="1000.0" lower="-0.04" upper="0.035" velocity="6.5"/>
   	<origin rpy="0 0 0" xyz="-0.015 0 0.0"/>
   	<parent link="arm_link_04"/>
-  	<child link="right_grip_link"/>
-  </joint>
-  <link name="left_grip_link">
-  	<inertial>
-  		<mass value="0.01"/>
-  		<origin xyz="0 0 0" rpy="0 0 0" />
-  		<inertia ixx="0.000010279" ixy="0" ixz="0" iyy="0.000010279" iyz="0" izz="0.000007225"/>
-  	</inertial>
-  	<collision>
-  	  <origin xyz="0.06 0.048 0.04" rpy="0 3.1415 -1.57"/>
-      <geometry>
-        <box size="0.06 0.02 0.08"/>
-      </geometry>
-  	</collision>
-  	<visual>
-  	  <origin xyz="0.06 0.048 0.04" rpy="0 3.1415 -1.57"/>
-      <geometry>
-        <box size="0.06 0.02 0.08"/>
-      </geometry>
-      <material name="white" />
-  	</visual>
-  </link>
-  <joint name="left_grip_joint" type="prismatic">
-  	<axis xyz="1 0 0"/>
-  	<limit effort="1000.0" upper="0.04" lower="-0.035" velocity="6.5"/>
-  	<origin rpy="0 0 0" xyz="-0.015 0 0.0"/>
-  	<parent link="arm_link_04"/>
-  	<child link="left_grip_link"/>
+  	<child link="grip_link"/>
   </joint>
 <transmission name="arm_joint_01_trans">
@@ -341,3 +314,13 @@
 </actuator>
 </transmission>
+<transmission name="grip_joint_trans">
+<type>transmission_interface/SimpleTransmission</type>
+<joint name="grip_joint">
+<hardwareInterface>hardware_interface/EffortJointInterface</hardwareInterface>
+</joint>
+<actuator name="motor5">
+<hardwareInterface>hardware_interface/EffortJointInterface</hardwareInterface>
+<mechanicalInterface>1</mechanicalInterface>
+</actuator>
+</transmission>
 </robot>

Commit message: TODO: same as previous commit

File: urdf/m2wr_arm.xacro (robot description, xacro)
@@ -254,5 +254,5 @@
   	</inertial>
   	<collision>
-  	  <origin xyz="-0.032 0.048 0.04" rpy="0 3.1415 -1.57"/>
+  	  <origin xyz="0 0.048 0.04" rpy="0 3.1415 -1.57"/>
       <geometry>
         <box size="0.06 0.02 0.08"/>
@@ -260,5 +260,5 @@
   	</collision>
   	<visual>
-  	  <origin xyz="-0.032 0.048 0.04" rpy="0 3.1415 -1.57"/>
+  	  <origin xyz="0 0.048 0.04" rpy="0 3.1415 -1.57"/>
       <geometry>
         <box size="0.06 0.02 0.08"/>

Commit message: It only remains the last arm and the gripper, then a bit of dimensions modifications

File: urdf/m2wr_arm.xacro (robot description, xacro)
@@ -17,5 +17,5 @@
               <origin rpy="0 1.5707 1.5707" xyz="0 0 0"/>
               <geometry>
-                <cylinder length="0.04" radius="0.1"/>
+                <cylinder length="0.04" radius="0.13"/>
               </geometry>
             </collision>
@@ -23,5 +23,5 @@
               <origin rpy="0 1.5707 1.5707" xyz="0 0 0"/>
               <geometry>
-                <cylinder length="0.04" radius="0.1"/>
+                <cylinder length="0.04" radius="0.13"/>
               </geometry>
             </visual>
@@ -42,11 +42,11 @@
     <pose>0 0 0.1 0 0 0</pose>
     <inertial>
-      <mass value="5"/>
-      <origin rpy="0 0 0" xyz="0 0 0.1"/>
+      <mass value="7"/>
+      <origin rpy="0 0 0" xyz="0 0 0.12"/>
       <inertia ixx="0.0395416666667" ixy="0" ixz="0" iyy="0.106208333333" iyz="0" izz="0.106208333333"/>
     </inertial>
     <collision name="collision_chassis">
       <geometry>
-        <box size="0.5 0.3 0.07"/>
+        <box size="0.8 0.6 0.08"/>
       </geometry>
     </collision>
@@ -54,5 +54,5 @@
       <origin rpy="0 0 0" xyz="0 0 0"/>
       <geometry>
-        <box size="0.5 0.3 0.07"/>
+        <box size="0.8 0.6 0.08"/>
       </geometry>
       <material name="blue"/>
@@ -60,7 +60,7 @@
     <!-- caster front -->
     <collision name="caster_front_collision">
-      <origin rpy=" 0 0 0" xyz="0.35 0 -0.05"/>
-      <geometry>
-        <sphere radius="0.05"/>
+      <origin rpy=" 0 0 0" xyz="0.4 0 -0.05"/>
+      <geometry>
+        <sphere radius="0.07"/>
       </geometry>
       <surface>
@@ -76,7 +76,7 @@
     </collision>
     <visual name="caster_front_visual">
-      <origin rpy=" 0 0 0" xyz="0.2 0 -0.05"/>
-      <geometry>
-        <sphere radius="0.05"/>
+      <origin rpy=" 0 0 0" xyz="0.4 0 -0.05"/>
+      <geometry>
+        <sphere radius="0.065"/>
       </geometry>
     </visual>
@@ -85,6 +85,6 @@
   <xacro:link_wheel name="link_right_wheel" />
   <xacro:link_wheel name="link_left_wheel" />
-  <xacro:joint_wheel name="joint_right_wheel"  child="link_right_wheel"  origin_xyz="-0.05 0.15 0"  />
-  <xacro:joint_wheel name="joint_left_wheel"   child="link_left_wheel"   origin_xyz="-0.05 -0.15 0"  />
+  <xacro:joint_wheel name="joint_right_wheel"  child="link_right_wheel"  origin_xyz="-0.15 0.3 0"  />
+  <xacro:joint_wheel name="joint_left_wheel"   child="link_left_wheel"   origin_xyz="-0.15 -0.3 0"  />
 <!-- Laser and Link Laser-->
    <link name="laser">
@@ -116,18 +116,18 @@
   <link name="arm_base_link">
   	<inertial>
-  		<mass value="0.1"/>
-  		<origin xyz="0 0 0" rpy="0 0 0" />
+  		<mass value="0.35"/>
+  		<origin xyz="0 0 0.085" rpy="0 0 0" />
   		<inertia ixx="0.0000416666667" ixy="0" ixz="0" iyy="0.0000416666667" iyz="0" izz="0.0000416666667"/>
   	</inertial>
   	<collision>
-  	  <origin xyz="0 0 0" rpy="0 0 0"/>
-      <geometry>
-        <box size="0.1 0.1 0.2"/>
-      </geometry>
-  	</collision>
-  	<visual>
-  	  <origin xyz="0 0 0" rpy="0 0 0"/>
-      <geometry>
-        <box size="0.1 0.1 0.2"/>
+  	  <origin xyz="0 0 0.085" rpy="0 0 0"/>
+      <geometry>
+        <box size="0.15 0.15 0.35"/>
+      </geometry>
+  	</collision>
+  	<visual>
+  	  <origin xyz="0 0 0.085" rpy="0 0 0"/>
+      <geometry>
+        <box size="0.15 0.15 0.35"/>
       </geometry>
       <material name="red" />
@@ -135,5 +135,5 @@
   </link>
   <joint name="arm_base_to_base" type="fixed">
-  	<origin rpy="0 0 0" xyz="0 0 0.085"/>
+  	<origin rpy="0 0 0" xyz="0 0 0.1"/>
   	<parent link="base_link"/>
   	<child link="arm_base_link"/>
@@ -141,5 +141,5 @@
   <link name="arm_link_01">
   	<inertial>
-  		<mass value="0.025"/>
+  		<mass value="0.05"/>
   		<origin xyz="0 0 0" rpy="0 0 0" />
   		<inertia ixx="0.000010279" ixy="0" ixz="0" iyy="0.000010279" iyz="0" izz="0.000007225"/>
@@ -148,5 +148,5 @@
   	  <origin xyz="0 0 0" rpy="0 0 0"/>
       <geometry>
-        <cylinder radius="0.04" length="0.08"/>
+        <cylinder radius="0.045" length="0.3"/>
       </geometry>
   	</collision>
@@ -154,5 +154,5 @@
   	  <origin xyz="0 0 0" rpy="0 0 0"/>
       <geometry>
-        <cylinder radius="0.04" length="0.08"/>
+        <cylinder radius="0.045" length="0.3"/>
       </geometry>
       <material name="red" />
@@ -162,5 +162,5 @@
   	<axis xyz="0 0 1"/>
   	<limit effort="1000.0" lower="-3.14" upper="3.14" velocity="0.2"/>
-  	<origin rpy="0 0 0" xyz="0 0 0.09"/>
+  	<origin rpy="0 0 0" xyz="0 0 0.275"/>
   	<parent link="arm_base_link"/>
   	<child link="arm_link_01"/>
@@ -168,18 +168,18 @@
     <link name="arm_link_02">
   	<inertial>
-  		<mass value="0.025"/>
+  		<mass value="0.03"/>
   		<origin xyz="0 0 0" rpy="0 0 0" />
   		<inertia ixx="0.000010279" ixy="0" ixz="0" iyy="0.000010279" iyz="0" izz="0.000007225"/>
   	</inertial>
   	<collision>
-  	  <origin xyz="0 0 0.04" rpy="0 0 0"/>
-      <geometry>
-        <cylinder radius="0.04" length="0.08"/>
-      </geometry>
-  	</collision>
-  	<visual>
-  	  <origin xyz="0 0 0.04" rpy="0 0 0"/>
-      <geometry>
-        <cylinder radius="0.04" length="0.08"/>
+  	  <origin xyz="0 0.01 0" rpy="0 0 0"/>
+      <geometry>
+        <cylinder radius="0.04" length="0.12"/>
+      </geometry>
+  	</collision>
+  	<visual>
+  	  <origin xyz="0 0.01 0" rpy="0 0 0"/>
+      <geometry>
+        <cylinder radius="0.04" length="0.12"/>
       </geometry>
       <material name="red" />
@@ -187,7 +187,7 @@
   </link>
   <joint name="arm_joint_02" type="revolute">
-  	<axis xyz="1 0 0"/>
+  	<axis xyz="-1 0 0"/>
   	<limit effort="1000.0" lower="-1.8" upper="1.8" velocity="0.2"/>
-  	<origin rpy="0 0 0" xyz="0 0 0.04"/>
+  	<origin rpy="0 0 0" xyz="0 0 0.175"/>
   	<parent link="arm_link_01"/>
   	<child link="arm_link_02"/>
@@ -196,17 +196,17 @@
   	<inertial>
   		<mass value="0.025"/>
-  		<origin xyz="0 0 0" rpy="0 0 0" />
-  		<inertia ixx="0.000010279" ixy="0" ixz="0" iyy="0.000010279" iyz="0" izz="0.000007225"/>
-  	</inertial>
-  	<collision>
-  	  <origin xyz="0 0 0.04" rpy="0 0 0"/>
-      <geometry>
-        <cylinder radius="0.04" length="0.08"/>
-      </geometry>
-  	</collision>
-  	<visual>
-  	  <origin xyz="0 0 0.04" rpy="0 0 0"/>
-      <geometry>
-        <cylinder radius="0.04" length="0.08"/>
+  		<origin xyz="0 0 0.15" rpy="0 0 0" />
+  		<inertia ixx="0.000010279" ixy="0" ixz="0" iyy="0.000010279" iyz="0" izz="0.000007225"/>
+  	</inertial>
+  	<collision>
+  	  <origin xyz="0 0 0.15" rpy="0 0 0"/>
+      <geometry>
+        <cylinder radius="0.04" length="0.4"/>
+      </geometry>
+  	</collision>
+  	<visual>
+  	  <origin xyz="0 0 0.15" rpy="0 0 0"/>
+      <geometry>
+        <cylinder radius="0.04" length="0.4"/>
       </geometry>
       <material name="red" />
@@ -214,7 +214,7 @@
   </link>
   <joint name="arm_joint_03" type="revolute">
-  	<axis xyz="1 0 0"/>
+  	<axis xyz="-1 0 0"/>
   	<limit effort="1000.0" lower="-1.8" upper="1.8" velocity="0.2"/>
-  	<origin rpy="0 0 0" xyz="0 0 0.08"/>
+  	<origin rpy="0 0 0" xyz="0 0 0"/>
   	<parent link="arm_link_02"/>
   	<child link="arm_link_03"/>
@@ -223,5 +223,5 @@
   	<inertial>
   		<mass value="0.025"/>
-  		<origin xyz="0 0 0" rpy="0 0 0" />
+  		<origin xyz="0 0 0.04" rpy="0 0 0" />
   		<inertia ixx="0.000010279" ixy="0" ixz="0" iyy="0.000010279" iyz="0" izz="0.000007225"/>
   	</inertial>
@@ -243,5 +243,5 @@
   	<axis xyz="1 0 0"/>
   	<limit effort="1000.0" lower="-1.8" upper="1.8" velocity="0.5"/>
-  	<origin rpy="0 0 0" xyz="0 0 0.08"/>
+  	<origin rpy="0 0 0" xyz="0 0 0"/>
   	<parent link="arm_link_03"/>
   	<child link="arm_link_04"/>

Commit message: control parameters need to be fixed

File: urdf/m2wr_arm.xacro (robot description, xacro)
@@ -42,5 +42,5 @@
     <pose>0 0 0.1 0 0 0</pose>
     <inertial>
-      <mass value="7"/>
+      <mass value="7.5"/>
       <origin rpy="0 0 0" xyz="0 0 0.12"/>
       <inertia ixx="0.0395416666667" ixy="0" ixz="0" iyy="0.106208333333" iyz="0" izz="0.106208333333"/>
@@ -60,7 +60,7 @@
     <!-- caster front -->
     <collision name="caster_front_collision">
-      <origin rpy=" 0 0 0" xyz="0.4 0 -0.05"/>
-      <geometry>
-        <sphere radius="0.07"/>
+      <origin rpy=" 0 0 0" xyz="0.325 0 -0.065"/>
+      <geometry>
+        <sphere radius="0.065"/>
       </geometry>
       <surface>
@@ -76,5 +76,5 @@
     </collision>
     <visual name="caster_front_visual">
-      <origin rpy=" 0 0 0" xyz="0.4 0 -0.05"/>
+      <origin rpy=" 0 0 0" xyz="0.325 0 -0.065"/>
       <geometry>
         <sphere radius="0.065"/>
@@ -85,6 +85,6 @@
   <xacro:link_wheel name="link_right_wheel" />
   <xacro:link_wheel name="link_left_wheel" />
-  <xacro:joint_wheel name="joint_right_wheel"  child="link_right_wheel"  origin_xyz="-0.15 0.3 0"  />
-  <xacro:joint_wheel name="joint_left_wheel"   child="link_left_wheel"   origin_xyz="-0.15 -0.3 0"  />
+  <xacro:joint_wheel name="joint_right_wheel"  child="link_right_wheel"  origin_xyz="-0.15 0.32 0"  />
+  <xacro:joint_wheel name="joint_left_wheel"   child="link_left_wheel"   origin_xyz="-0.15 -0.32 0"  />
 <!-- Laser and Link Laser-->
    <link name="laser">
@@ -109,5 +109,5 @@
   </link>
   <joint name="joint_laser" type="fixed">
-    <origin xyz="0.15 0 0.05" rpy="0 0 0"/>
+    <origin xyz="0.3 0 0.05" rpy="0 0 0"/>
     <parent link="base_link"/>
     <child link="laser"/>
@@ -123,5 +123,5 @@
   	  <origin xyz="0 0 0.085" rpy="0 0 0"/>
       <geometry>
-        <box size="0.15 0.15 0.35"/>
+        <box size="0.18 0.18 0.35"/>
       </geometry>
   	</collision>
@@ -129,5 +129,5 @@
   	  <origin xyz="0 0 0.085" rpy="0 0 0"/>
       <geometry>
-        <box size="0.15 0.15 0.35"/>
+        <box size="0.18 0.18 0.35"/>
       </geometry>
       <material name="red" />
@@ -135,5 +135,5 @@
   </link>
   <joint name="arm_base_to_base" type="fixed">
-  	<origin rpy="0 0 0" xyz="0 0 0.1"/>
+  	<origin rpy="0 0 0" xyz="0 0 0.135"/>
   	<parent link="base_link"/>
   	<child link="arm_base_link"/>
@@ -162,5 +162,5 @@
   	<axis xyz="0 0 1"/>
   	<limit effort="1000.0" lower="-3.14" upper="3.14" velocity="0.2"/>
-  	<origin rpy="0 0 0" xyz="0 0 0.275"/>
+  	<origin rpy="0 0 1" xyz="0 0 0.35"/>
   	<parent link="arm_base_link"/>
   	<child link="arm_link_01"/>
@@ -175,5 +175,5 @@
   	  <origin xyz="0 0.01 0" rpy="0 0 0"/>
       <geometry>
-        <cylinder radius="0.04" length="0.12"/>
+        <cylinder radius="0.04" length="0.15"/>
       </geometry>
   	</collision>
@@ -181,5 +181,5 @@
   	  <origin xyz="0 0.01 0" rpy="0 0 0"/>
       <geometry>
-        <cylinder radius="0.04" length="0.12"/>
+        <cylinder radius="0.04" length="0.15"/>
       </geometry>
       <material name="red" />
@@ -187,7 +187,7 @@
   </link>
   <joint name="arm_joint_02" type="revolute">
-  	<axis xyz="-1 0 0"/>
+  	<axis xyz="1 0 0"/>
   	<limit effort="1000.0" lower="-1.8" upper="1.8" velocity="0.2"/>
-  	<origin rpy="0 0 0" xyz="0 0 0.175"/>
+  	<origin rpy="1.57 0 0" xyz="0 0 0.18"/>
   	<parent link="arm_link_01"/>
   	<child link="arm_link_02"/>
@@ -195,5 +195,5 @@
       <link name="arm_link_03">
   	<inertial>
-  		<mass value="0.025"/>
+  		<mass value="0.02"/>
   		<origin xyz="0 0 0.15" rpy="0 0 0" />
   		<inertia ixx="0.000010279" ixy="0" ixz="0" iyy="0.000010279" iyz="0" izz="0.000007225"/>
@@ -202,5 +202,5 @@
   	  <origin xyz="0 0 0.15" rpy="0 0 0"/>
       <geometry>
-        <cylinder radius="0.04" length="0.4"/>
+        <cylinder radius="0.037" length="0.4"/>
       </geometry>
   	</collision>
@@ -208,5 +208,5 @@
   	  <origin xyz="0 0 0.15" rpy="0 0 0"/>
       <geometry>
-        <cylinder radius="0.04" length="0.4"/>
+        <cylinder radius="0.037" length="0.4"/>
       </geometry>
       <material name="red" />
@@ -216,5 +216,5 @@
   	<axis xyz="-1 0 0"/>
   	<limit effort="1000.0" lower="-1.8" upper="1.8" velocity="0.2"/>
-  	<origin rpy="0 0 0" xyz="0 0 0"/>
+  	<origin rpy="-1.57 0 0" xyz="0 0 0"/>
   	<parent link="arm_link_02"/>
   	<child link="arm_link_03"/>
@@ -222,5 +222,5 @@
     <link name="arm_link_04">
   	<inertial>
-  		<mass value="0.025"/>
+  		<mass value="0.018"/>
   		<origin xyz="0 0 0.04" rpy="0 0 0" />
   		<inertia ixx="0.000010279" ixy="0" ixz="0" iyy="0.000010279" iyz="0" izz="0.000007225"/>
@@ -243,5 +243,5 @@
   	<axis xyz="1 0 0"/>
   	<limit effort="1000.0" lower="-1.8" upper="1.8" velocity="0.5"/>
-  	<origin rpy="0 0 0" xyz="0 0 0"/>
+  	<origin rpy="0 0 3.14" xyz="0 0 0.355"/>
   	<parent link="arm_link_03"/>
   	<child link="arm_link_04"/>
@@ -249,5 +249,5 @@
 <link name="grip_link">
   	<inertial>
-  		<mass value="0.01"/>
+  		<mass value="0.008"/>
   		<origin xyz="0 0 0" rpy="0 0 0" />
   		<inertia ixx="0.000010279" ixy="0" ixz="0" iyy="0.000010279" iyz="0" izz="0.000007225"/>
@@ -270,5 +270,5 @@
   	<axis xyz="1 0 0"/>
   	<limit effort="1000.0" lower="-0.04" upper="0.035" velocity="6.5"/>
-  	<origin rpy="0 0 0" xyz="-0.015 0 0.0"/>
+  	<origin rpy="0 0 0" xyz="0 0 0"/>
   	<parent link="arm_link_04"/>
   	<child link="grip_link"/>
