Commit message: generated moveit package in order to control the robot, now it must be considered the fact  that the robot does not work as expected and so on

File: urdf/m2wr_arm.xacro (robot description, xacro)
@@ -123,5 +123,5 @@
   	  <origin xyz="0 0 0.085" rpy="0 0 0"/>
       <geometry>
-        <box size="0.18 0.18 0.35"/>
+        <box size="0.18 0.18 0.45"/>
       </geometry>
   	</collision>
@@ -129,5 +129,5 @@
   	  <origin xyz="0 0 0.085" rpy="0 0 0"/>
       <geometry>
-        <box size="0.18 0.18 0.35"/>
+        <box size="0.18 0.18 0.45"/>
       </geometry>
       <material name="red" />
@@ -135,5 +135,5 @@
   </link>
   <joint name="arm_base_to_base" type="fixed">
-  	<origin rpy="0 0 0" xyz="0 0 0.135"/>
+  	<origin rpy="0 0 0" xyz="0 0 0.14"/>
   	<parent link="base_link"/>
   	<child link="arm_base_link"/>
@@ -141,5 +141,5 @@
   <link name="arm_link_01">
   	<inertial>
-  		<mass value="0.05"/>
+  		<mass value="0.045"/>
   		<origin xyz="0 0 0" rpy="0 0 0" />
   		<inertia ixx="0.000010279" ixy="0" ixz="0" iyy="0.000010279" iyz="0" izz="0.000007225"/>
@@ -148,5 +148,5 @@
   	  <origin xyz="0 0 0" rpy="0 0 0"/>
       <geometry>
-        <cylinder radius="0.045" length="0.3"/>
+        <cylinder radius="0.045" length="0.35"/>
       </geometry>
   	</collision>
@@ -154,5 +154,5 @@
   	  <origin xyz="0 0 0" rpy="0 0 0"/>
       <geometry>
-        <cylinder radius="0.045" length="0.3"/>
+        <cylinder radius="0.045" length="0.35"/>
       </geometry>
       <material name="red" />
@@ -161,6 +161,6 @@
   <joint name="arm_joint_01" type="revolute">
   	<axis xyz="0 0 1"/>
-  	<limit effort="1000.0" lower="-3.14" upper="3.14" velocity="0.2"/>
-  	<origin rpy="0 0 1" xyz="0 0 0.35"/>
+  	<limit effort="1000.0" lower="-3.14" upper="3.14" velocity="0.5"/>
+  	<origin rpy="0 0 -1" xyz="0 0 0.4"/>
   	<parent link="arm_base_link"/>
   	<child link="arm_link_01"/>
@@ -168,5 +168,5 @@
     <link name="arm_link_02">
   	<inertial>
-  		<mass value="0.03"/>
+  		<mass value="0.025"/>
   		<origin xyz="0 0 0" rpy="0 0 0" />
   		<inertia ixx="0.000010279" ixy="0" ixz="0" iyy="0.000010279" iyz="0" izz="0.000007225"/>
@@ -175,5 +175,5 @@
   	  <origin xyz="0 0.01 0" rpy="0 0 0"/>
       <geometry>
-        <cylinder radius="0.04" length="0.15"/>
+        <cylinder radius="0.04" length="0.175"/>
       </geometry>
   	</collision>
@@ -181,5 +181,5 @@
   	  <origin xyz="0 0.01 0" rpy="0 0 0"/>
       <geometry>
-        <cylinder radius="0.04" length="0.15"/>
+        <cylinder radius="0.04" length="0.175"/>
       </geometry>
       <material name="red" />
@@ -188,5 +188,5 @@
   <joint name="arm_joint_02" type="revolute">
   	<axis xyz="1 0 0"/>
-  	<limit effort="1000.0" lower="-1.8" upper="1.8" velocity="0.2"/>
+  	<limit effort="1000.0" lower="-1.8" upper="1.8" velocity="0.3"/>
   	<origin rpy="1.57 0 0" xyz="0 0 0.18"/>
   	<parent link="arm_link_01"/>
@@ -195,5 +195,5 @@
       <link name="arm_link_03">
   	<inertial>
-  		<mass value="0.02"/>
+  		<mass value="0.015"/>
   		<origin xyz="0 0 0.15" rpy="0 0 0" />
   		<inertia ixx="0.000010279" ixy="0" ixz="0" iyy="0.000010279" iyz="0" izz="0.000007225"/>
@@ -215,5 +215,5 @@
   <joint name="arm_joint_03" type="revolute">
   	<axis xyz="-1 0 0"/>
-  	<limit effort="1000.0" lower="-1.8" upper="1.8" velocity="0.2"/>
+  	<limit effort="1000.0" lower="-1.8" upper="1.8" velocity="0.3"/>
   	<origin rpy="-1.57 0 0" xyz="0 0 0"/>
   	<parent link="arm_link_02"/>
@@ -222,5 +222,5 @@
     <link name="arm_link_04">
   	<inertial>
-  		<mass value="0.018"/>
+  		<mass value="0.0125"/>
   		<origin xyz="0 0 0.04" rpy="0 0 0" />
   		<inertia ixx="0.000010279" ixy="0" ixz="0" iyy="0.000010279" iyz="0" izz="0.000007225"/>
@@ -242,6 +242,6 @@
   <joint name="arm_joint_04" type="revolute">
   	<axis xyz="1 0 0"/>
-  	<limit effort="1000.0" lower="-1.8" upper="1.8" velocity="0.5"/>
-  	<origin rpy="0 0 3.14" xyz="0 0 0.355"/>
+  	<limit effort="1000.0" lower="-1.8" upper="1.8" velocity="0.75"/>
+  	<origin rpy="0 0 0" xyz="0 0 0.355"/>
   	<parent link="arm_link_03"/>
   	<child link="arm_link_04"/>
@@ -249,5 +249,5 @@
 <link name="grip_link">
   	<inertial>
-  		<mass value="0.008"/>
+  		<mass value="0.0075"/>
   		<origin xyz="0 0 0" rpy="0 0 0" />
   		<inertia ixx="0.000010279" ixy="0" ixz="0" iyy="0.000010279" iyz="0" izz="0.000007225"/>

File: urdf/robot6.urdf (robot description, URDF)
Before this commit: robot m2wr, 11 links, 10 joints
Links:
- removed link left_grip_link
- removed link right_grip_link
- added link grip_link, mass 0.0075; collision box size=0.06 0.02 0.08; visual box size=0.06 0.02 0.08
- link arm_base_link: mass 0.1 -> 0.35; geometry collision box size=0.18 0.18 0.45; visual box size=0.18 0.18 0.45
- link arm_link_01: mass 0.025 -> 0.045; geometry collision cylinder length=0.35 radius=0.045; visual cylinder length=0.35 radius=0.045
- link arm_link_02: geometry collision cylinder length=0.175 radius=0.04; visual cylinder length=0.175 radius=0.04
- link arm_link_03: mass 0.025 -> 0.015; geometry collision cylinder length=0.4 radius=0.037; visual cylinder length=0.4 radius=0.037
- link arm_link_04: mass 0.025 -> 0.0125
- link base_link: mass 5 -> 7.5; geometry collision box size=0.8 0.6 0.08; collision sphere radius=0.065
- link link_left_wheel: geometry collision cylinder length=0.04 radius=0.13; visual cylinder length=0.04 radius=0.13
- link link_right_wheel: geometry collision cylinder length=0.04 radius=0.13; visual cylinder length=0.04 radius=0.13
Joints:
- removed joint left_grip_joint
- removed joint right_grip_joint
- added joint grip_joint: type prismatic, parent arm_link_04, child grip_link, origin xyz=0 0 0 rpy=0 0 0, axis 1 0 0, limit lower=-0.04 upper=0.035 effort=1000.0 velocity=6.5
- joint arm_base_to_base: origin xyz=0 0 0.085 rpy=0 0 0 -> xyz=0 0 0.14 rpy=0 0 0
- joint arm_joint_01: limit lower=-3.14 upper=3.14 effort=1000.0 velocity=0.2 -> lower=-3.14 upper=3.14 effort=1000.0 velocity=0.5; origin xyz=0 0 0.09 rpy=0 0 0 -> xyz=0 0 0.4 rpy=0 0 -1
- joint arm_joint_02: limit lower=-1.8 upper=1.8 effort=1000.0 velocity=0.2 -> lower=-1.8 upper=1.8 effort=1000.0 velocity=0.3; origin xyz=0 0 0.04 rpy=0 0 0 -> xyz=0 0 0.18 rpy=1.57 0 0
- joint arm_joint_03: axis 1 0 0 -> -1 0 0; limit lower=-1.8 upper=1.8 effort=1000.0 velocity=0.2 -> lower=-1.8 upper=1.8 effort=1000.0 velocity=0.3; origin xyz=0 0 0.08 rpy=0 0 0 -> xyz=0 0 0 rpy=-1.57 0 0
- joint arm_joint_04: limit lower=-1.8 upper=1.8 effort=1000.0 velocity=0.5 -> lower=-1.8 upper=1.8 effort=1000.0 velocity=0.75; origin xyz=0 0 0.08 rpy=0 0 0 -> xyz=0 0 0.355 rpy=0 0 0
- joint joint_laser: origin xyz=0.15 0 0.05 rpy=0 0 0 -> xyz=0.3 0 0.05 rpy=0 0 0
- joint joint_left_wheel: origin xyz=-0.05 -0.15 0 rpy=0 0 0 -> xyz=-0.15 -0.32 0 rpy=0 0 0
- joint joint_right_wheel: origin xyz=-0.05 0.15 0 rpy=0 0 0 -> xyz=-0.15 0.32 0 rpy=0 0 0

Commit message: robot model fine tuned, notice that with moveit robot in gazebo does not move

File: urdf/m2wr_arm.xacro (robot description, xacro)
@@ -187,5 +187,5 @@
   </link>
   <joint name="arm_joint_02" type="revolute">
-  	<axis xyz="1 0 0"/>
+  	<axis xyz="0 0 1"/>
   	<limit effort="1000.0" lower="-1.8" upper="1.8" velocity="0.3"/>
   	<origin rpy="1.57 0 0" xyz="0 0 0.18"/>
@@ -214,5 +214,5 @@
   </link>
   <joint name="arm_joint_03" type="revolute">
-  	<axis xyz="-1 0 0"/>
+  	<axis xyz="0 0 1"/>
   	<limit effort="1000.0" lower="-1.8" upper="1.8" velocity="0.3"/>
   	<origin rpy="-1.57 0 0" xyz="0 0 0"/>

Commit message: error, grip must be renamed cluedo since the assignment needs it

File: urdf/m2wr_arm.xacro (robot description, xacro)
@@ -247,5 +247,5 @@
   	<child link="arm_link_04"/>
   </joint>
-<link name="grip_link">
+<link name="cluedo_link">
   	<inertial>
   		<mass value="0.0075"/>
@@ -267,10 +267,10 @@
   	</visual>
   </link>
-  <joint name="grip_joint" type="prismatic">
+  <joint name="cluedo_joint" type="prismatic">
   	<axis xyz="1 0 0"/>
   	<limit effort="1000.0" lower="-0.04" upper="0.035" velocity="6.5"/>
   	<origin rpy="0 0 0" xyz="0 0 0"/>
   	<parent link="arm_link_04"/>
-  	<child link="grip_link"/>
+  	<child link="cluedo_link"/>
   </joint>
 <transmission name="arm_joint_01_trans">
@@ -314,7 +314,7 @@
 </actuator>
 </transmission>
-<transmission name="grip_joint_trans">
-<type>transmission_interface/SimpleTransmission</type>
-<joint name="grip_joint">
+<transmission name="cluedo_joint_trans">
+<type>transmission_interface/SimpleTransmission</type>
+<joint name="cluedo_joint">
 <hardwareInterface>hardware_interface/EffortJointInterface</hardwareInterface>
 </joint>

File: urdf/robot6.urdf (robot description, URDF)
Before this commit: robot m2wr, 10 links, 9 joints
Links:
- removed link grip_link
- added link cluedo_link, mass 0.0075; collision box size=0.06 0.02 0.08; visual box size=0.06 0.02 0.08
Joints:
- removed joint grip_joint
- added joint cluedo_joint: type prismatic, parent arm_link_04, child cluedo_link, origin xyz=0 0 0 rpy=0 0 0, axis 1 0 0, limit lower=-0.04 upper=0.035 effort=1000.0 velocity=6.5

Commit message: replan and target received does not work

File: urdf/m2wr_arm.xacro (robot description, xacro)
@@ -123,5 +123,5 @@
   	  <origin xyz="0 0 0.085" rpy="0 0 0"/>
       <geometry>
-        <box size="0.18 0.18 0.45"/>
+        <box size="0.18 0.18 0.47"/>
       </geometry>
   	</collision>
@@ -129,5 +129,5 @@
   	  <origin xyz="0 0 0.085" rpy="0 0 0"/>
       <geometry>
-        <box size="0.18 0.18 0.45"/>
+        <box size="0.18 0.18 0.47"/>
       </geometry>
       <material name="red" />
@@ -148,5 +148,5 @@
   	  <origin xyz="0 0 0" rpy="0 0 0"/>
       <geometry>
-        <cylinder radius="0.045" length="0.35"/>
+        <cylinder radius="0.045" length="0.38"/>
       </geometry>
   	</collision>
@@ -154,5 +154,5 @@
   	  <origin xyz="0 0 0" rpy="0 0 0"/>
       <geometry>
-        <cylinder radius="0.045" length="0.35"/>
+        <cylinder radius="0.045" length="0.38"/>
       </geometry>
       <material name="red" />
@@ -175,5 +175,5 @@
   	  <origin xyz="0 0.01 0" rpy="0 0 0"/>
       <geometry>
-        <cylinder radius="0.04" length="0.175"/>
+        <cylinder radius="0.04" length="0.2"/>
       </geometry>
   	</collision>
@@ -181,5 +181,5 @@
   	  <origin xyz="0 0.01 0" rpy="0 0 0"/>
       <geometry>
-        <cylinder radius="0.04" length="0.175"/>
+        <cylinder radius="0.04" length="0.2"/>
       </geometry>
       <material name="red" />
@@ -196,5 +196,5 @@
   	<inertial>
   		<mass value="0.015"/>
-  		<origin xyz="0 0 0.15" rpy="0 0 0" />
+  		<origin xyz="0 0 0.175" rpy="0 0 0" />
   		<inertia ixx="0.000010279" ixy="0" ixz="0" iyy="0.000010279" iyz="0" izz="0.000007225"/>
   	</inertial>
@@ -202,5 +202,5 @@
   	  <origin xyz="0 0 0.15" rpy="0 0 0"/>
       <geometry>
-        <cylinder radius="0.037" length="0.4"/>
+        <cylinder radius="0.037" length="0.62"/>
       </geometry>
   	</collision>
@@ -208,5 +208,5 @@
   	  <origin xyz="0 0 0.15" rpy="0 0 0"/>
       <geometry>
-        <cylinder radius="0.037" length="0.4"/>
+        <cylinder radius="0.037" length="0.62"/>
       </geometry>
       <material name="red" />
@@ -243,5 +243,5 @@
   	<axis xyz="1 0 0"/>
   	<limit effort="1000.0" lower="-1.8" upper="1.8" velocity="0.75"/>
-  	<origin rpy="0 0 0" xyz="0 0 0.355"/>
+  	<origin rpy="0 0 0" xyz="0 0 0.45"/>
   	<parent link="arm_link_03"/>
   	<child link="arm_link_04"/>

File: urdf/robot6.urdf (robot description, URDF)
Before this commit: robot m2wr, 10 links, 9 joints
Links:
- link arm_base_link: geometry collision box size=0.18 0.18 0.47; visual box size=0.18 0.18 0.47
- link arm_link_01: geometry collision cylinder length=0.38 radius=0.045; visual cylinder length=0.38 radius=0.045
- link arm_link_02: geometry collision cylinder length=0.2 radius=0.04; visual cylinder length=0.2 radius=0.04
- link arm_link_03: geometry collision cylinder length=0.62 radius=0.037; visual cylinder length=0.62 radius=0.037
Joints:
- joint arm_joint_04: origin xyz=0 0 0.355 rpy=0 0 0 -> xyz=0 0 0.45 rpy=0 0 0

Commit message: last 'working' package

File: urdf/m2wr_arm.xacro (robot description, xacro)
@@ -121,5 +121,5 @@
   	</inertial>
   	<collision>
-  	  <origin xyz="0 0 0.085" rpy="0 0 0"/>
+  	  <origin xyz="0 0 0.088" rpy="0 0 0"/>
       <geometry>
         <box size="0.18 0.18 0.47"/>
@@ -127,5 +127,5 @@
   	</collision>
   	<visual>
-  	  <origin xyz="0 0 0.085" rpy="0 0 0"/>
+  	  <origin xyz="0 0 0.088" rpy="0 0 0"/>
       <geometry>
         <box size="0.18 0.18 0.47"/>
@@ -202,5 +202,5 @@
   	  <origin xyz="0 0 0.15" rpy="0 0 0"/>
       <geometry>
-        <cylinder radius="0.037" length="0.62"/>
+        <cylinder radius="0.036" length="0.65"/>
       </geometry>
   	</collision>
@@ -208,5 +208,5 @@
   	  <origin xyz="0 0 0.15" rpy="0 0 0"/>
       <geometry>
-        <cylinder radius="0.037" length="0.62"/>
+        <cylinder radius="0.036" length="0.65"/>
       </geometry>
       <material name="red" />

File: urdf/robot6.urdf (robot description, URDF)
Before this commit: robot m2wr, 10 links, 9 joints
Links:
- link arm_link_03: geometry collision cylinder length=0.65 radius=0.036; visual cylinder length=0.65 radius=0.036

Commit message: now the robot is a 6 dof and may be somehow reach the target. In order to better undertsand this there must be other tests. In addition, replanning always fail

File: urdf/m2wr_arm.xacro (robot description, xacro)
@@ -117,9 +117,9 @@
   	<inertial>
   		<mass value="0.35"/>
-  		<origin xyz="0 0 0.085" rpy="0 0 0" />
+  		<origin xyz="0 0 0.085" rpy="0 1.57 0" />
   		<inertia ixx="0.0000416666667" ixy="0" ixz="0" iyy="0.0000416666667" iyz="0" izz="0.0000416666667"/>
   	</inertial>
   	<collision>
-  	  <origin xyz="0 0 0.088" rpy="0 0 0"/>
+  	  <origin xyz="0 0 0.088" rpy="0 1.57 0"/>
       <geometry>
         <box size="0.18 0.18 0.47"/>
@@ -127,5 +127,5 @@
   	</collision>
   	<visual>
-  	  <origin xyz="0 0 0.088" rpy="0 0 0"/>
+  	  <origin xyz="0 0 0.088" rpy="0 1.57 0"/>
       <geometry>
         <box size="0.18 0.18 0.47"/>
@@ -134,6 +134,7 @@
   	</visual>
   </link>
-  <joint name="arm_base_to_base" type="fixed">
-  	<origin rpy="0 0 0" xyz="0 0 0.14"/>
+  <joint name="arm_base_to_base" type="prismatic">
+    <limit effort="1000.0" lower="0" upper="0.25" velocity="2"/>
+  	<origin rpy="0 -1.57 0" xyz="0 0 0.15"/>
   	<parent link="base_link"/>
   	<child link="arm_base_link"/>
@@ -162,5 +163,5 @@
   	<axis xyz="0 0 1"/>
   	<limit effort="1000.0" lower="-3.14" upper="3.14" velocity="0.5"/>
-  	<origin rpy="0 0 -1" xyz="0 0 0.4"/>
+  	<origin rpy="0 1.57 0" xyz="0.4 0 0.1"/>
   	<parent link="arm_base_link"/>
   	<child link="arm_link_01"/>
@@ -274,4 +275,14 @@
   	<child link="cluedo_link"/>
   </joint>
+<transmission name="arm_joint_base_trans">
+<type>transmission_interface/SimpleTransmission</type>
+<joint name="arm_base_to_base">
+<hardwareInterface>hardware_interface/EffortJointInterface</hardwareInterface>
+</joint>
+<actuator name="motor0">
+<hardwareInterface>hardware_interface/EffortJointInterface</hardwareInterface>
+<mechanicalInterface>1</mechanicalInterface>
+</actuator>
+</transmission>
 <transmission name="arm_joint_01_trans">
 <type>transmission_interface/SimpleTransmission</type>

File: urdf/robot6.urdf (robot description, URDF)
Before this commit: robot m2wr, 10 links, 9 joints
Joints:
- joint arm_base_to_base: limit (none) -> lower=0 upper=0.25 effort=1000.0 velocity=2; origin xyz=0 0 0.14 rpy=0 0 0 -> xyz=0 0 0.15 rpy=0 -1.57 0; type fixed -> prismatic
- joint arm_joint_01: origin xyz=0 0 0.4 rpy=0 0 -1 -> xyz=0.4 0 0.1 rpy=0 1.57 0

Commit message: TODO: fix replanning, implement investigation

File: urdf/m2wr_arm.xacro (robot description, xacro)
@@ -149,5 +149,5 @@
   	  <origin xyz="0 0 0" rpy="0 0 0"/>
       <geometry>
-        <cylinder radius="0.045" length="0.38"/>
+        <cylinder radius="0.045" length="0.4"/>
       </geometry>
   	</collision>
@@ -155,5 +155,5 @@
   	  <origin xyz="0 0 0" rpy="0 0 0"/>
       <geometry>
-        <cylinder radius="0.045" length="0.38"/>
+        <cylinder radius="0.045" length="0.4"/>
       </geometry>
       <material name="red" />
@@ -197,17 +197,17 @@
   	<inertial>
   		<mass value="0.015"/>
-  		<origin xyz="0 0 0.175" rpy="0 0 0" />
-  		<inertia ixx="0.000010279" ixy="0" ixz="0" iyy="0.000010279" iyz="0" izz="0.000007225"/>
-  	</inertial>
-  	<collision>
-  	  <origin xyz="0 0 0.15" rpy="0 0 0"/>
-      <geometry>
-        <cylinder radius="0.036" length="0.65"/>
-      </geometry>
-  	</collision>
-  	<visual>
-  	  <origin xyz="0 0 0.15" rpy="0 0 0"/>
-      <geometry>
-        <cylinder radius="0.036" length="0.65"/>
+  		<origin xyz="0 0 0.21" rpy="0 0 0" />
+  		<inertia ixx="0.000010279" ixy="0" ixz="0" iyy="0.000010279" iyz="0" izz="0.000007225"/>
+  	</inertial>
+  	<collision>
+  	  <origin xyz="0 0 0.21" rpy="0 0 0"/>
+      <geometry>
+        <cylinder radius="0.036" length="0.67"/>
+      </geometry>
+  	</collision>
+  	<visual>
+  	  <origin xyz="0 0 0.21" rpy="0 0 0"/>
+      <geometry>
+        <cylinder radius="0.036" length="0.67"/>
       </geometry>
       <material name="red" />
@@ -244,5 +244,5 @@
   	<axis xyz="1 0 0"/>
   	<limit effort="1000.0" lower="-1.8" upper="1.8" velocity="0.75"/>
-  	<origin rpy="0 0 0" xyz="0 0 0.45"/>
+  	<origin rpy="0 0 0" xyz="0 0 0.55"/>
   	<parent link="arm_link_03"/>
   	<child link="arm_link_04"/>

File: urdf/robot6.urdf (robot description, URDF)
Before this commit: robot m2wr, 10 links, 9 joints
Links:
- link arm_link_01: geometry collision cylinder length=0.4 radius=0.045; visual cylinder length=0.4 radius=0.045
- link arm_link_03: geometry collision cylinder length=0.67 radius=0.036; visual cylinder length=0.67 radius=0.036
Joints:
- joint arm_joint_04: origin xyz=0 0 0.45 rpy=0 0 0 -> xyz=0 0 0.55 rpy=0 0 0

Commit message: sometimes find hint fails in finding hint. replanning fails also.

File: urdf/m2wr_arm.xacro (robot description, xacro)
@@ -135,5 +135,5 @@
   </link>
   <joint name="arm_base_to_base" type="prismatic">
-    <limit effort="1000.0" lower="0" upper="0.25" velocity="2"/>
+    <limit effort="1000.0" lower="0" upper="0.27" velocity="2"/>
   	<origin rpy="0 -1.57 0" xyz="0 0 0.15"/>
   	<parent link="base_link"/>
@@ -203,5 +203,5 @@
   	  <origin xyz="0 0 0.21" rpy="0 0 0"/>
       <geometry>
-        <cylinder radius="0.036" length="0.67"/>
+        <cylinder radius="0.036" length="0.7"/>
       </geometry>
   	</collision>
@@ -209,5 +209,5 @@
   	  <origin xyz="0 0 0.21" rpy="0 0 0"/>
       <geometry>
-        <cylinder radius="0.036" length="0.67"/>
+        <cylinder radius="0.036" length="0.7"/>
       </geometry>
       <material name="red" />
@@ -244,5 +244,5 @@
   	<axis xyz="1 0 0"/>
   	<limit effort="1000.0" lower="-1.8" upper="1.8" velocity="0.75"/>
-  	<origin rpy="0 0 0" xyz="0 0 0.55"/>
+  	<origin rpy="0 0 0" xyz="0 0 0.57"/>
   	<parent link="arm_link_03"/>
   	<child link="arm_link_04"/>

File: urdf/robot6.urdf (robot description, URDF)
Before this commit: robot m2wr, 10 links, 9 joints
Links:
- link arm_link_03: geometry collision cylinder length=0.7 radius=0.036; visual cylinder length=0.7 radius=0.036
Joints:
- joint arm_base_to_base: limit lower=0 upper=0.25 effort=1000.0 velocity=2 -> lower=0 upper=0.27 effort=1000.0 velocity=2
- joint arm_joint_04: origin xyz=0 0 0.55 rpy=0 0 0 -> xyz=0 0 0.57 rpy=0 0 0

Commit message: still same problems as before, but the execution of the planning and some other adjustments have been done

File: urdf/m2wr_arm.xacro (robot description, xacro)
@@ -197,9 +197,9 @@
   	<inertial>
   		<mass value="0.015"/>
-  		<origin xyz="0 0 0.21" rpy="0 0 0" />
-  		<inertia ixx="0.000010279" ixy="0" ixz="0" iyy="0.000010279" iyz="0" izz="0.000007225"/>
-  	</inertial>
-  	<collision>
-  	  <origin xyz="0 0 0.21" rpy="0 0 0"/>
+  		<origin xyz="0 0 0.3" rpy="0 0 0" />
+  		<inertia ixx="0.000010279" ixy="0" ixz="0" iyy="0.000010279" iyz="0" izz="0.000007225"/>
+  	</inertial>
+  	<collision>
+  	  <origin xyz="0 0 0.3" rpy="0 0 0"/>
       <geometry>
         <cylinder radius="0.036" length="0.7"/>
@@ -207,5 +207,5 @@
   	</collision>
   	<visual>
-  	  <origin xyz="0 0 0.21" rpy="0 0 0"/>
+  	  <origin xyz="0 0 0.3" rpy="0 0 0"/>
       <geometry>
         <cylinder radius="0.036" length="0.7"/>
@@ -224,9 +224,9 @@
   	<inertial>
   		<mass value="0.0125"/>
-  		<origin xyz="0 0 0.04" rpy="0 0 0" />
-  		<inertia ixx="0.000010279" ixy="0" ixz="0" iyy="0.000010279" iyz="0" izz="0.000007225"/>
-  	</inertial>
-  	<collision>
-  	  <origin xyz="0 0 0.04" rpy="0 0 1.57"/>
+  		<origin xyz="0 0 0.045" rpy="0 0 0" />
+  		<inertia ixx="0.000010279" ixy="0" ixz="0" iyy="0.000010279" iyz="0" izz="0.000007225"/>
+  	</inertial>
+  	<collision>
+  	  <origin xyz="0 0 0.045" rpy="0 0 1.57"/>
       <geometry>
         <box size="0.034 0.2 0.08"/>
@@ -234,5 +234,5 @@
   	</collision>
   	<visual>
-  	  <origin xyz="0 0 0.04" rpy="0 0 1.57"/>
+  	  <origin xyz="0 0 0.045" rpy="0 0 1.57"/>
       <geometry>
         <box size="0.034 0.2 0.08"/>
@@ -244,5 +244,5 @@
   	<axis xyz="1 0 0"/>
   	<limit effort="1000.0" lower="-1.8" upper="1.8" velocity="0.75"/>
-  	<origin rpy="0 0 0" xyz="0 0 0.57"/>
+  	<origin rpy="0 0 0" xyz="0 0 0.65"/>
   	<parent link="arm_link_03"/>
   	<child link="arm_link_04"/>

File: urdf/robot6.urdf (robot description, URDF)
Before this commit: robot m2wr, 10 links, 9 joints
Joints:
- joint arm_joint_04: origin xyz=0 0 0.57 rpy=0 0 0 -> xyz=0 0 0.65 rpy=0 0 0
