Commit message: trying to solve moveit issues

File: urdf/m2wr_arm.xacro (robot description, xacro)
@@ -149,5 +149,5 @@
   	  <origin xyz="0 0 0" rpy="0 0 0"/>
       <geometry>
-        <cylinder radius="0.045" length="0.4"/>
+        <cylinder radius="0.045" length="0.7"/>
       </geometry>
   	</collision>
@@ -155,5 +155,5 @@
   	  <origin xyz="0 0 0" rpy="0 0 0"/>
       <geometry>
-        <cylinder radius="0.045" length="0.4"/>
+        <cylinder radius="0.045" length="0.7"/>
       </geometry>
       <material name="red" />
@@ -163,5 +163,5 @@
   	<axis xyz="0 0 1"/>
   	<limit effort="1000.0" lower="-3.14" upper="3.14" velocity="0.5"/>
-  	<origin rpy="0 1.57 0" xyz="0.4 0 0.1"/>
+  	<origin rpy="0 1.57 0" xyz="0.48 0 0.1"/>
   	<parent link="arm_base_link"/>
   	<child link="arm_link_01"/>
@@ -174,5 +174,5 @@
   	</inertial>
   	<collision>
-  	  <origin xyz="0 0.01 0" rpy="0 0 0"/>
+  	  <origin xyz="0 0 0" rpy="0 0 0"/>
       <geometry>
         <cylinder radius="0.04" length="0.2"/>
@@ -180,5 +180,5 @@
   	</collision>
   	<visual>
-  	  <origin xyz="0 0.01 0" rpy="0 0 0"/>
+  	  <origin xyz="0 0 0" rpy="0 0 0"/>
       <geometry>
         <cylinder radius="0.04" length="0.2"/>
@@ -189,6 +189,6 @@
   <joint name="arm_joint_02" type="revolute">
   	<axis xyz="0 0 1"/>
-  	<limit effort="1000.0" lower="-1.8" upper="1.8" velocity="0.3"/>
-  	<origin rpy="1.57 0 0" xyz="0 0 0.18"/>
+  	<limit effort="1000.0" lower="-3.14" upper="3.14" velocity="0.3"/>
+  	<origin rpy="1.57 0 0" xyz="0 0 0.35"/>
   	<parent link="arm_link_01"/>
   	<child link="arm_link_02"/>
@@ -196,18 +196,18 @@
       <link name="arm_link_03">
   	<inertial>
-  		<mass value="0.015"/>
-  		<origin xyz="0 0 0.3" rpy="0 0 0" />
-  		<inertia ixx="0.000010279" ixy="0" ixz="0" iyy="0.000010279" iyz="0" izz="0.000007225"/>
-  	</inertial>
-  	<collision>
-  	  <origin xyz="0 0 0.3" rpy="0 0 0"/>
-      <geometry>
-        <cylinder radius="0.036" length="0.7"/>
-      </geometry>
-  	</collision>
-  	<visual>
-  	  <origin xyz="0 0 0.3" rpy="0 0 0"/>
-      <geometry>
-        <cylinder radius="0.036" length="0.7"/>
+  		<mass value="0.01"/>
+  		<origin xyz="0 0 0.38" rpy="0 0 0" />
+  		<inertia ixx="0.000010279" ixy="0" ixz="0" iyy="0.000010279" iyz="0" izz="0.000007225"/>
+  	</inertial>
+  	<collision>
+  	  <origin xyz="0 0 0.38" rpy="0 0 0"/>
+      <geometry>
+        <cylinder radius="0.035" length="0.8"/>
+      </geometry>
+  	</collision>
+  	<visual>
+  	  <origin xyz="0 0 0.38" rpy="0 0 0"/>
+      <geometry>
+        <cylinder radius="0.035" length="0.8"/>
       </geometry>
       <material name="red" />
@@ -216,5 +216,5 @@
   <joint name="arm_joint_03" type="revolute">
   	<axis xyz="0 0 1"/>
-  	<limit effort="1000.0" lower="-1.8" upper="1.8" velocity="0.3"/>
+  	<limit effort="1000.0" lower="-3.14" upper="3.14" velocity="0.3"/>
   	<origin rpy="-1.57 0 0" xyz="0 0 0"/>
   	<parent link="arm_link_02"/>
@@ -243,6 +243,6 @@
   <joint name="arm_joint_04" type="revolute">
   	<axis xyz="1 0 0"/>
-  	<limit effort="1000.0" lower="-1.8" upper="1.8" velocity="0.75"/>
-  	<origin rpy="0 0 0" xyz="0 0 0.65"/>
+  	<limit effort="1000.0" lower="-3.14" upper="3.14" velocity="0.75"/>
+  	<origin rpy="0 0 0" xyz="0 0 0.75"/>
   	<parent link="arm_link_03"/>
   	<child link="arm_link_04"/>

File: urdf/robot6.urdf (robot description, URDF)
Before this commit: robot m2wr, 10 links, 9 joints
Links:
- link arm_link_01: geometry collision cylinder length=0.7 radius=0.045; visual cylinder length=0.7 radius=0.045
- link arm_link_03: mass 0.015 -> 0.01; geometry collision cylinder length=0.8 radius=0.035; visual cylinder length=0.8 radius=0.035
Joints:
- joint arm_joint_01: origin xyz=0.4 0 0.1 rpy=0 1.57 0 -> xyz=0.48 0 0.1 rpy=0 1.57 0
- joint arm_joint_02: limit lower=-1.8 upper=1.8 effort=1000.0 velocity=0.3 -> lower=-3.14 upper=3.14 effort=1000.0 velocity=0.3; origin xyz=0 0 0.18 rpy=1.57 0 0 -> xyz=0 0 0.35 rpy=1.57 0 0
- joint arm_joint_03: limit lower=-1.8 upper=1.8 effort=1000.0 velocity=0.3 -> lower=-3.14 upper=3.14 effort=1000.0 velocity=0.3
- joint arm_joint_04: limit lower=-1.8 upper=1.8 effort=1000.0 velocity=0.75 -> lower=-3.14 upper=3.14 effort=1000.0 velocity=0.75; origin xyz=0 0 0.65 rpy=0 0 0 -> xyz=0 0 0.75 rpy=0 0 0

Commit message: improvements and well performing robot until some time

File: urdf/m2wr_arm.xacro (robot description, xacro)
@@ -42,5 +42,5 @@
     <pose>0 0 0.1 0 0 0</pose>
     <inertial>
-      <mass value="7.5"/>
+      <mass value="8.5"/>
       <origin rpy="0 0 0" xyz="0 0 0.12"/>
       <inertia ixx="0.0395416666667" ixy="0" ixz="0" iyy="0.106208333333" iyz="0" izz="0.106208333333"/>
@@ -135,5 +135,5 @@
   </link>
   <joint name="arm_base_to_base" type="prismatic">
-    <limit effort="1000.0" lower="0" upper="0.27" velocity="2"/>
+    <limit effort="1000.0" lower="0" upper="0.32" velocity="2"/>
   	<origin rpy="0 -1.57 0" xyz="0 0 0.15"/>
   	<parent link="base_link"/>
@@ -149,5 +149,5 @@
   	  <origin xyz="0 0 0" rpy="0 0 0"/>
       <geometry>
-        <cylinder radius="0.045" length="0.7"/>
+        <cylinder radius="0.045" length="0.6"/>
       </geometry>
   	</collision>
@@ -155,5 +155,5 @@
   	  <origin xyz="0 0 0" rpy="0 0 0"/>
       <geometry>
-        <cylinder radius="0.045" length="0.7"/>
+        <cylinder radius="0.045" length="0.6"/>
       </geometry>
       <material name="red" />
@@ -162,5 +162,5 @@
   <joint name="arm_joint_01" type="revolute">
   	<axis xyz="0 0 1"/>
-  	<limit effort="1000.0" lower="-3.14" upper="3.14" velocity="0.5"/>
+  	<limit effort="1000.0" lower="-6.28" upper="6.28" velocity="0.5"/>
   	<origin rpy="0 1.57 0" xyz="0.48 0 0.1"/>
   	<parent link="arm_base_link"/>
@@ -176,5 +176,5 @@
   	  <origin xyz="0 0 0" rpy="0 0 0"/>
       <geometry>
-        <cylinder radius="0.04" length="0.2"/>
+        <cylinder radius="0.04" length="0.6"/>
       </geometry>
   	</collision>
@@ -182,5 +182,5 @@
   	  <origin xyz="0 0 0" rpy="0 0 0"/>
       <geometry>
-        <cylinder radius="0.04" length="0.2"/>
+        <cylinder radius="0.04" length="0.6"/>
       </geometry>
       <material name="red" />
@@ -189,6 +189,6 @@
   <joint name="arm_joint_02" type="revolute">
   	<axis xyz="0 0 1"/>
-  	<limit effort="1000.0" lower="-3.14" upper="3.14" velocity="0.3"/>
-  	<origin rpy="1.57 0 0" xyz="0 0 0.35"/>
+  	<limit effort="1000.0" lower="-6.28" upper="6.28" velocity="0.3"/>
+  	<origin rpy="1.57 0 0" xyz="0 0.3 0.3"/>
   	<parent link="arm_link_01"/>
   	<child link="arm_link_02"/>
@@ -196,5 +196,5 @@
       <link name="arm_link_03">
   	<inertial>
-  		<mass value="0.01"/>
+  		<mass value="0.008"/>
   		<origin xyz="0 0 0.38" rpy="0 0 0" />
   		<inertia ixx="0.000010279" ixy="0" ixz="0" iyy="0.000010279" iyz="0" izz="0.000007225"/>
@@ -203,5 +203,5 @@
   	  <origin xyz="0 0 0.38" rpy="0 0 0"/>
       <geometry>
-        <cylinder radius="0.035" length="0.8"/>
+        <cylinder radius="0.035" length="0.68"/>
       </geometry>
   	</collision>
@@ -209,5 +209,5 @@
   	  <origin xyz="0 0 0.38" rpy="0 0 0"/>
       <geometry>
-        <cylinder radius="0.035" length="0.8"/>
+        <cylinder radius="0.035" length="0.68"/>
       </geometry>
       <material name="red" />
@@ -216,6 +216,6 @@
   <joint name="arm_joint_03" type="revolute">
   	<axis xyz="0 0 1"/>
-  	<limit effort="1000.0" lower="-3.14" upper="3.14" velocity="0.3"/>
-  	<origin rpy="-1.57 0 0" xyz="0 0 0"/>
+  	<limit effort="1000.0" lower="-6.28" upper="6.28" velocity="0.3"/>
+  	<origin rpy="-1.57 0 0" xyz="0 0 -0.25"/>
   	<parent link="arm_link_02"/>
   	<child link="arm_link_03"/>
@@ -223,5 +223,5 @@
     <link name="arm_link_04">
   	<inertial>
-  		<mass value="0.0125"/>
+  		<mass value="0.007"/>
   		<origin xyz="0 0 0.045" rpy="0 0 0" />
   		<inertia ixx="0.000010279" ixy="0" ixz="0" iyy="0.000010279" iyz="0" izz="0.000007225"/>
@@ -243,6 +243,6 @@
   <joint name="arm_joint_04" type="revolute">
   	<axis xyz="1 0 0"/>
-  	<limit effort="1000.0" lower="-3.14" upper="3.14" velocity="0.75"/>
-  	<origin rpy="0 0 0" xyz="0 0 0.75"/>
+  	<limit effort="1000.0" lower="-6.28" upper="6.28" velocity="0.75"/>
+  	<origin rpy="0 0 0" xyz="0 0 0.7"/>
   	<parent link="arm_link_03"/>
   	<child link="arm_link_04"/>
@@ -250,5 +250,5 @@
 <link name="cluedo_link">
   	<inertial>
-  		<mass value="0.0075"/>
+  		<mass value="0.007"/>
   		<origin xyz="0 0 0" rpy="0 0 0" />
   		<inertia ixx="0.000010279" ixy="0" ixz="0" iyy="0.000010279" iyz="0" izz="0.000007225"/>

File: urdf/robot6.urdf (robot description, URDF)
Before this commit: robot m2wr, 10 links, 9 joints
Links:
- link arm_link_01: geometry collision cylinder length=0.6 radius=0.045; visual cylinder length=0.6 radius=0.045
- link arm_link_02: geometry collision cylinder length=0.6 radius=0.04; visual cylinder length=0.6 radius=0.04
- link arm_link_03: mass 0.01 -> 0.008; geometry collision cylinder length=0.68 radius=0.035; visual cylinder length=0.68 radius=0.035
- link arm_link_04: mass 0.0125 -> 0.007
- link base_link: mass 7.5 -> 8.5
- link cluedo_link: mass 0.0075 -> 0.007
Joints:
- joint arm_base_to_base: limit lower=0 upper=0.27 effort=1000.0 velocity=2 -> lower=0 upper=0.32 effort=1000.0 velocity=2
- joint arm_joint_01: limit lower=-3.14 upper=3.14 effort=1000.0 velocity=0.5 -> lower=-6.28 upper=6.28 effort=1000.0 velocity=0.5
- joint arm_joint_02: limit lower=-3.14 upper=3.14 effort=1000.0 velocity=0.3 -> lower=-6.28 upper=6.28 effort=1000.0 velocity=0.3; origin xyz=0 0 0.35 rpy=1.57 0 0 -> xyz=0 0.3 0.3 rpy=1.57 0 0
- joint arm_joint_03: limit lower=-3.14 upper=3.14 effort=1000.0 velocity=0.3 -> lower=-6.28 upper=6.28 effort=1000.0 velocity=0.3; origin xyz=0 0 0 rpy=-1.57 0 0 -> xyz=0 0 -0.25 rpy=-1.57 0 0
- joint arm_joint_04: limit lower=-3.14 upper=3.14 effort=1000.0 velocity=0.75 -> lower=-6.28 upper=6.28 effort=1000.0 velocity=0.75; origin xyz=0 0 0.75 rpy=0 0 0 -> xyz=0 0 0.7 rpy=0 0 0

Commit message: MISSING: reason, oracle, documentation, a bit of navigation and user interface

File: urdf/m2wr_arm.xacro (robot description, xacro)
@@ -135,5 +135,5 @@
   </link>
   <joint name="arm_base_to_base" type="prismatic">
-    <limit effort="1000.0" lower="0" upper="0.32" velocity="2"/>
+    <limit effort="1000.0" lower="0" upper="0.32" velocity="2.2"/>
   	<origin rpy="0 -1.57 0" xyz="0 0 0.15"/>
   	<parent link="base_link"/>
@@ -149,5 +149,5 @@
   	  <origin xyz="0 0 0" rpy="0 0 0"/>
       <geometry>
-        <cylinder radius="0.045" length="0.6"/>
+        <cylinder radius="0.045" length="0.36"/>
       </geometry>
   	</collision>
@@ -155,5 +155,5 @@
   	  <origin xyz="0 0 0" rpy="0 0 0"/>
       <geometry>
-        <cylinder radius="0.045" length="0.6"/>
+        <cylinder radius="0.045" length="0.36"/>
       </geometry>
       <material name="red" />
@@ -162,6 +162,6 @@
   <joint name="arm_joint_01" type="revolute">
   	<axis xyz="0 0 1"/>
-  	<limit effort="1000.0" lower="-6.28" upper="6.28" velocity="0.5"/>
-  	<origin rpy="0 1.57 0" xyz="0.48 0 0.1"/>
+  	<limit effort="1000.0" lower="-6.28" upper="6.28" velocity="0.55"/>
+  	<origin rpy="0 1.57 0" xyz="0.28 0 0.1"/>
   	<parent link="arm_base_link"/>
   	<child link="arm_link_01"/>
@@ -176,5 +176,5 @@
   	  <origin xyz="0 0 0" rpy="0 0 0"/>
       <geometry>
-        <cylinder radius="0.04" length="0.6"/>
+        <cylinder radius="0.04" length="0.5"/>
       </geometry>
   	</collision>
@@ -182,5 +182,5 @@
   	  <origin xyz="0 0 0" rpy="0 0 0"/>
       <geometry>
-        <cylinder radius="0.04" length="0.6"/>
+        <cylinder radius="0.04" length="0.5"/>
       </geometry>
       <material name="red" />
@@ -189,6 +189,6 @@
   <joint name="arm_joint_02" type="revolute">
   	<axis xyz="0 0 1"/>
-  	<limit effort="1000.0" lower="-6.28" upper="6.28" velocity="0.3"/>
-  	<origin rpy="1.57 0 0" xyz="0 0.3 0.3"/>
+  	<limit effort="1000.0" lower="-6.28" upper="6.28" velocity="0.4"/>
+  	<origin rpy="2 0 0" xyz="0 0.17 0.3"/>
   	<parent link="arm_link_01"/>
   	<child link="arm_link_02"/>
@@ -197,17 +197,17 @@
   	<inertial>
   		<mass value="0.008"/>
-  		<origin xyz="0 0 0.38" rpy="0 0 0" />
-  		<inertia ixx="0.000010279" ixy="0" ixz="0" iyy="0.000010279" iyz="0" izz="0.000007225"/>
-  	</inertial>
-  	<collision>
-  	  <origin xyz="0 0 0.38" rpy="0 0 0"/>
-      <geometry>
-        <cylinder radius="0.035" length="0.68"/>
-      </geometry>
-  	</collision>
-  	<visual>
-  	  <origin xyz="0 0 0.38" rpy="0 0 0"/>
-      <geometry>
-        <cylinder radius="0.035" length="0.68"/>
+  		<origin xyz="0 0 0.32" rpy="0 0 0" />
+  		<inertia ixx="0.000010279" ixy="0" ixz="0" iyy="0.000010279" iyz="0" izz="0.000007225"/>
+  	</inertial>
+  	<collision>
+  	  <origin xyz="0 0 0.32" rpy="0 0 0"/>
+      <geometry>
+        <cylinder radius="0.035" length="0.55"/>
+      </geometry>
+  	</collision>
+  	<visual>
+  	  <origin xyz="0 0 0.32" rpy="0 0 0"/>
+      <geometry>
+        <cylinder radius="0.035" length="0.55"/>
       </geometry>
       <material name="red" />
@@ -216,6 +216,6 @@
   <joint name="arm_joint_03" type="revolute">
   	<axis xyz="0 0 1"/>
-  	<limit effort="1000.0" lower="-6.28" upper="6.28" velocity="0.3"/>
-  	<origin rpy="-1.57 0 0" xyz="0 0 -0.25"/>
+  	<limit effort="1000.0" lower="-6.28" upper="6.28" velocity="0.4"/>
+  	<origin rpy="-1.57 0 0" xyz="0 0 -0.22"/>
   	<parent link="arm_link_02"/>
   	<child link="arm_link_03"/>
@@ -224,9 +224,9 @@
   	<inertial>
   		<mass value="0.007"/>
-  		<origin xyz="0 0 0.045" rpy="0 0 0" />
-  		<inertia ixx="0.000010279" ixy="0" ixz="0" iyy="0.000010279" iyz="0" izz="0.000007225"/>
-  	</inertial>
-  	<collision>
-  	  <origin xyz="0 0 0.045" rpy="0 0 1.57"/>
+  		<origin xyz="0 0 0.047" rpy="0 0 0" />
+  		<inertia ixx="0.000010279" ixy="0" ixz="0" iyy="0.000010279" iyz="0" izz="0.000007225"/>
+  	</inertial>
+  	<collision>
+  	  <origin xyz="0 0 0.047" rpy="0 0 1.57"/>
       <geometry>
         <box size="0.034 0.2 0.08"/>
@@ -234,5 +234,5 @@
   	</collision>
   	<visual>
-  	  <origin xyz="0 0 0.045" rpy="0 0 1.57"/>
+  	  <origin xyz="0 0 0.047" rpy="0 0 1.57"/>
       <geometry>
         <box size="0.034 0.2 0.08"/>
@@ -243,6 +243,6 @@
   <joint name="arm_joint_04" type="revolute">
   	<axis xyz="1 0 0"/>
-  	<limit effort="1000.0" lower="-6.28" upper="6.28" velocity="0.75"/>
-  	<origin rpy="0 0 0" xyz="0 0 0.7"/>
+  	<limit effort="1000.0" lower="-6.28" upper="6.28" velocity="0.77"/>
+  	<origin rpy="0 0 0" xyz="0 0 0.58"/>
   	<parent link="arm_link_03"/>
   	<child link="arm_link_04"/>
@@ -270,5 +270,5 @@
   <joint name="cluedo_joint" type="prismatic">
   	<axis xyz="1 0 0"/>
-  	<limit effort="1000.0" lower="-0.04" upper="0.035" velocity="6.5"/>
+  	<limit effort="1000.0" lower="-0.04" upper="0.035" velocity="6.6"/>
   	<origin rpy="0 0 0" xyz="0 0 0"/>
   	<parent link="arm_link_04"/>

File: urdf/robot6.urdf (robot description, URDF)
Before this commit: robot m2wr, 10 links, 9 joints
Links:
- link arm_link_01: geometry collision cylinder length=0.36 radius=0.045; visual cylinder length=0.36 radius=0.045
- link arm_link_02: geometry collision cylinder length=0.5 radius=0.04; visual cylinder length=0.5 radius=0.04
- link arm_link_03: geometry collision cylinder length=0.55 radius=0.035; visual cylinder length=0.55 radius=0.035
Joints:
- joint arm_base_to_base: limit lower=0 upper=0.32 effort=1000.0 velocity=2 -> lower=0 upper=0.32 effort=1000.0 velocity=2.2
- joint arm_joint_01: limit lower=-6.28 upper=6.28 effort=1000.0 velocity=0.5 -> lower=-6.28 upper=6.28 effort=1000.0 velocity=0.55; origin xyz=0.48 0 0.1 rpy=0 1.57 0 -> xyz=0.28 0 0.1 rpy=0 1.57 0
- joint arm_joint_02: limit lower=-6.28 upper=6.28 effort=1000.0 velocity=0.3 -> lower=-6.28 upper=6.28 effort=1000.0 velocity=0.4; origin xyz=0 0.3 0.3 rpy=1.57 0 0 -> xyz=0 0.17 0.3 rpy=2 0 0
- joint arm_joint_03: limit lower=-6.28 upper=6.28 effort=1000.0 velocity=0.3 -> lower=-6.28 upper=6.28 effort=1000.0 velocity=0.4; origin xyz=0 0 -0.25 rpy=-1.57 0 0 -> xyz=0 0 -0.22 rpy=-1.57 0 0
- joint arm_joint_04: limit lower=-6.28 upper=6.28 effort=1000.0 velocity=0.75 -> lower=-6.28 upper=6.28 effort=1000.0 velocity=0.77; origin xyz=0 0 0.7 rpy=0 0 0 -> xyz=0 0 0.58 rpy=0 0 0
- joint cluedo_joint: limit lower=-0.04 upper=0.035 effort=1000.0 velocity=6.5 -> lower=-0.04 upper=0.035 effort=1000.0 velocity=6.6

Commit message: Some tests must be made. But meanwhile comments and documentation started

File: urdf/m2wr_arm.xacro (robot description, xacro)
@@ -42,5 +42,5 @@
     <pose>0 0 0.1 0 0 0</pose>
     <inertial>
-      <mass value="8.5"/>
+      <mass value="9"/>
       <origin rpy="0 0 0" xyz="0 0 0.12"/>
       <inertia ixx="0.0395416666667" ixy="0" ixz="0" iyy="0.106208333333" iyz="0" izz="0.106208333333"/>
@@ -48,5 +48,5 @@
     <collision name="collision_chassis">
       <geometry>
-        <box size="0.8 0.6 0.08"/>
+        <box size="0.8 0.5 0.08"/>
       </geometry>
     </collision>
@@ -54,5 +54,5 @@
       <origin rpy="0 0 0" xyz="0 0 0"/>
       <geometry>
-        <box size="0.8 0.6 0.08"/>
+        <box size="0.8 0.5 0.08"/>
       </geometry>
       <material name="blue"/>
@@ -85,6 +85,6 @@
   <xacro:link_wheel name="link_right_wheel" />
   <xacro:link_wheel name="link_left_wheel" />
-  <xacro:joint_wheel name="joint_right_wheel"  child="link_right_wheel"  origin_xyz="-0.15 0.32 0"  />
-  <xacro:joint_wheel name="joint_left_wheel"   child="link_left_wheel"   origin_xyz="-0.15 -0.32 0"  />
+  <xacro:joint_wheel name="joint_right_wheel"  child="link_right_wheel"  origin_xyz="-0.15 0.27 0"  />
+  <xacro:joint_wheel name="joint_left_wheel"   child="link_left_wheel"   origin_xyz="-0.15 -0.27 0"  />
 <!-- Laser and Link Laser-->
    <link name="laser">
@@ -135,5 +135,5 @@
   </link>
   <joint name="arm_base_to_base" type="prismatic">
-    <limit effort="1000.0" lower="0" upper="0.32" velocity="2.2"/>
+    <limit effort="1000.0" lower="0" upper="0.32" velocity="1.5"/>
   	<origin rpy="0 -1.57 0" xyz="0 0 0.15"/>
   	<parent link="base_link"/>

File: urdf/robot6.urdf (robot description, URDF)
Before this commit: robot m2wr, 10 links, 9 joints
Links:
- link base_link: mass 8.5 -> 9; geometry collision box size=0.8 0.5 0.08; collision sphere radius=0.065
Joints:
- joint arm_base_to_base: limit lower=0 upper=0.32 effort=1000.0 velocity=2.2 -> lower=0 upper=0.32 effort=1000.0 velocity=1.5
- joint joint_left_wheel: origin xyz=-0.15 -0.32 0 rpy=0 0 0 -> xyz=-0.15 -0.27 0 rpy=0 0 0
- joint joint_right_wheel: origin xyz=-0.15 0.32 0 rpy=0 0 0 -> xyz=-0.15 0.27 0 rpy=0 0 0

Commit message: some adjustents have been made. But seems there is a problem with the reason part

File: urdf/m2wr_arm.xacro (robot description, xacro)
@@ -91,5 +91,5 @@
     <inertial>
       <origin xyz="0 0 0" rpy="0 0 0" />
-      <mass value="1" />
+      <mass value="1.2" />
       <xacro:cylinder_inertia mass="1" r="0.05" l="0.1" />
     </inertial>

File: urdf/robot6.urdf (robot description, URDF)
Before this commit: robot m2wr, 10 links, 9 joints
Links:
- link laser: mass 1 -> 1.2

Commit message: adding markers, moveit, movebase

File: urdf/m2wr_arm.xacro (robot description, xacro)
@@ -275,4 +275,32 @@
   	<child link="cluedo_link"/>
   </joint>
+  <link name="camera_link">
+	    <collision>
+	      <origin xyz="0 0 0.025" rpy="0 0 0"/>
+	      <geometry>
+		<box size="0.05 0.05 0.05"/>
+	      </geometry>
+	    </collision>
+	    <visual>
+	      <origin xyz="0 0 0.025" rpy="0 0 0"/>
+	      <geometry>
+		<box size="0.05 0.05 0.05"/>
+	      </geometry>
+	      <material name="red">
+		<color rgba="1 0 0 1"/>
+	      </material>
+	    </visual>
+	    <inertial>
+	      <mass value="1e-5" />
+	      <origin xyz="0 0 0" rpy="0 0 0"/>
+	      <inertia ixx="1e-6" ixy="0" ixz="0" iyy="1e-6" iyz="0" izz="1e-6" />
+	    </inertial>
+  </link>
+  <joint name="camera_joint" type="fixed">
+	    <axis xyz="0 1 0" />
+	    <origin xyz="0 0 0.05" rpy="0 0 0"/>
+	    <parent link="cluedo_link"/>
+	    <child link="camera_link"/>
+	 </joint>
 <transmission name="arm_joint_base_trans">
 <type>transmission_interface/SimpleTransmission</type>

Commit message: written navigation node, hope it will work. Now it is the turn of Investigation node

File: urdf/m2wr_arm.xacro (robot description, xacro)
@@ -299,5 +299,5 @@
   <joint name="camera_joint" type="fixed">
 	    <axis xyz="0 1 0" />
-	    <origin xyz="0 0 0.05" rpy="0 0 0"/>
+	    <origin xyz="0 0.1 0.02" rpy="0 0 0"/>
 	    <parent link="cluedo_link"/>
 	    <child link="camera_link"/>

File: urdf/robot6.urdf (robot description, URDF)
Before this commit: robot m2wr, 10 links, 9 joints
Links:
- added link camera_link, mass 1e-5; collision box size=0.05 0.05 0.05; visual box size=0.05 0.05 0.05
Joints:
- added joint camera_joint: type fixed, parent cluedo_link, child camera_link, origin xyz=0 0.1 0.02 rpy=0 0 0, axis 0 1 0
