Commit message: now slam gmapping seems to work: parameters must be optimized

File: urdf/m2wr_arm.xacro (robot description, xacro)
@@ -7,5 +7,5 @@
                 iyy="${mass*(3*r*r+l*l)/12}" iyz = "0" izz="${mass*(r*r)/2}" />
  </xacro:macro>
-    <xacro:macro name="link_wheel" params="name">
+   <xacro:macro name="link_wheel" params="name">
         <link name="${name}">
             <inertial>
@@ -17,5 +17,5 @@
               <origin rpy="0 1.5707 1.5707" xyz="0 0 0"/>
               <geometry>
-                <cylinder length="0.04" radius="0.13"/>
+                <cylinder length="0.04" radius="0.1"/>
               </geometry>
             </collision>
@@ -23,5 +23,5 @@
               <origin rpy="0 1.5707 1.5707" xyz="0 0 0"/>
               <geometry>
-                <cylinder length="0.04" radius="0.13"/>
+                <cylinder length="0.04" radius="0.1"/>
               </geometry>
             </visual>
@@ -42,11 +42,11 @@
     <pose>0 0 0.1 0 0 0</pose>
     <inertial>
-      <mass value="9"/>
-      <origin rpy="0 0 0" xyz="0 0 0.12"/>
+      <mass value="10"/>
+      <origin rpy="0 0 0" xyz="0 0 0.1"/>
       <inertia ixx="0.0395416666667" ixy="0" ixz="0" iyy="0.106208333333" iyz="0" izz="0.106208333333"/>
     </inertial>
     <collision name="collision_chassis">
       <geometry>
-        <box size="0.8 0.5 0.08"/>
+        <box size="0.5 0.3 0.07"/>
       </geometry>
     </collision>
@@ -54,5 +54,5 @@
       <origin rpy="0 0 0" xyz="0 0 0"/>
       <geometry>
-        <box size="0.8 0.5 0.08"/>
+        <box size="0.5 0.3 0.07"/>
       </geometry>
       <material name="blue"/>
@@ -60,7 +60,7 @@
     <!-- caster front -->
     <collision name="caster_front_collision">
-      <origin rpy=" 0 0 0" xyz="0.325 0 -0.065"/>
-      <geometry>
-        <sphere radius="0.065"/>
+      <origin rpy=" 0 0 0" xyz="0.35 0 -0.05"/>
+      <geometry>
+        <sphere radius="0.05"/>
       </geometry>
       <surface>
@@ -76,7 +76,7 @@
     </collision>
     <visual name="caster_front_visual">
-      <origin rpy=" 0 0 0" xyz="0.325 0 -0.065"/>
-      <geometry>
-        <sphere radius="0.065"/>
+      <origin rpy=" 0 0 0" xyz="0.2 0 -0.05"/>
+      <geometry>
+        <sphere radius="0.05"/>
       </geometry>
     </visual>
@@ -85,6 +85,6 @@
   <xacro:link_wheel name="link_right_wheel" />
   <xacro:link_wheel name="link_left_wheel" />
-  <xacro:joint_wheel name="joint_right_wheel"  child="link_right_wheel"  origin_xyz="-0.15 0.27 0"  />
-  <xacro:joint_wheel name="joint_left_wheel"   child="link_left_wheel"   origin_xyz="-0.15 -0.27 0"  />
+  <xacro:joint_wheel name="joint_right_wheel"  child="link_right_wheel"  origin_xyz="-0.05 -0.15 0"  />
+  <xacro:joint_wheel name="joint_left_wheel"   child="link_left_wheel"   origin_xyz="-0.05 0.15 0"  />
 <!-- Laser and Link Laser-->
    <link name="laser">
@@ -123,11 +123,11 @@
   	  <origin xyz="0 0 0.088" rpy="0 1.57 0"/>
       <geometry>
-        <box size="0.18 0.18 0.47"/>
-      </geometry>
-  	</collision>
-  	<visual>
-  	  <origin xyz="0 0 0.088" rpy="0 1.57 0"/>
-      <geometry>
-        <box size="0.18 0.18 0.47"/>
+        <box size="0.12 0.12 0.47"/>
+      </geometry>
+  	</collision>
+  	<visual>
+  	  <origin xyz="0 0 0.085" rpy="0 1.57 0"/>
+      <geometry>
+        <box size="0.12 0.12 0.47"/>
       </geometry>
       <material name="red" />
@@ -136,5 +136,5 @@
   <joint name="arm_base_to_base" type="prismatic">
     <limit effort="1000.0" lower="0" upper="0.32" velocity="1.5"/>
-  	<origin rpy="0 -1.57 0" xyz="0 0 0.15"/>
+  	<origin rpy="0 -1.57 0" xyz="0 0 0.17"/>
   	<parent link="base_link"/>
   	<child link="arm_base_link"/>
@@ -293,5 +293,5 @@
 	    <inertial>
 	      <mass value="1e-5" />
-	      <origin xyz="0 0 0" rpy="0 0 0"/>
+	      <origin xyz="0 0 0.025" rpy="0 0 0"/>
 	      <inertia ixx="1e-6" ixy="0" ixz="0" iyy="1e-6" iyz="0" izz="1e-6" />
 	    </inertial>
@@ -299,5 +299,5 @@
   <joint name="camera_joint" type="fixed">
 	    <axis xyz="0 1 0" />
-	    <origin xyz="0 0.1 0.02" rpy="0 0 0"/>
+	    <origin xyz="0 0.1 0.02" rpy="0 0 1.57"/>
 	    <parent link="cluedo_link"/>
 	    <child link="camera_link"/>

File: urdf/robot6.urdf (robot description, URDF)
Before this commit: robot m2wr, 11 links, 10 joints
Links:
- link arm_base_link: geometry collision box size=0.12 0.12 0.47; visual box size=0.12 0.12 0.47
- link base_link: mass 9 -> 10; geometry collision box size=0.5 0.3 0.07; collision sphere radius=0.05
- link link_left_wheel: geometry collision cylinder length=0.04 radius=0.1; visual cylinder length=0.04 radius=0.1
- link link_right_wheel: geometry collision cylinder length=0.04 radius=0.1; visual cylinder length=0.04 radius=0.1
Joints:
- joint arm_base_to_base: origin xyz=0 0 0.15 rpy=0 -1.57 0 -> xyz=0 0 0.17 rpy=0 -1.57 0
- joint camera_joint: origin xyz=0 0.1 0.02 rpy=0 0 0 -> xyz=0 0.1 0.02 rpy=0 0 1.57
- joint joint_left_wheel: origin xyz=-0.15 -0.27 0 rpy=0 0 0 -> xyz=-0.05 0.15 0 rpy=0 0 0
- joint joint_right_wheel: origin xyz=-0.15 0.27 0 rpy=0 0 0 -> xyz=-0.05 -0.15 0 rpy=0 0 0

Commit message: b

File: urdf/m2wr_arm.xacro (robot description, xacro)
@@ -10,5 +10,5 @@
         <link name="${name}">
             <inertial>
-              <mass value="0.2"/>
+              <mass value="0.8"/>
               <origin rpy="0 1.5707 1.5707" xyz="0 0 0"/>
               <inertia ixx="0.000526666666667" ixy="0" ixz="0" iyy="0.000526666666667" iyz="0" izz="0.001"/>
@@ -42,5 +42,5 @@
     <pose>0 0 0.1 0 0 0</pose>
     <inertial>
-      <mass value="10"/>
+      <mass value="12"/>
       <origin rpy="0 0 0" xyz="0 0 0.1"/>
       <inertia ixx="0.0395416666667" ixy="0" ixz="0" iyy="0.106208333333" iyz="0" izz="0.106208333333"/>
@@ -48,5 +48,5 @@
     <collision name="collision_chassis">
       <geometry>
-        <box size="0.5 0.3 0.07"/>
+        <box size="0.5 0.4 0.07"/>
       </geometry>
     </collision>
@@ -54,5 +54,5 @@
       <origin rpy="0 0 0" xyz="0 0 0"/>
       <geometry>
-        <box size="0.5 0.3 0.07"/>
+        <box size="0.5 0.4 0.07"/>
       </geometry>
       <material name="blue"/>
@@ -85,12 +85,12 @@
   <xacro:link_wheel name="link_right_wheel" />
   <xacro:link_wheel name="link_left_wheel" />
-  <xacro:joint_wheel name="joint_right_wheel"  child="link_right_wheel"  origin_xyz="-0.05 -0.15 0"  />
-  <xacro:joint_wheel name="joint_left_wheel"   child="link_left_wheel"   origin_xyz="-0.05 0.15 0"  />
+  <xacro:joint_wheel name="joint_right_wheel"  child="link_right_wheel"  origin_xyz="-0.05 -0.22 0"  />
+  <xacro:joint_wheel name="joint_left_wheel"   child="link_left_wheel"   origin_xyz="-0.05 0.22 0"  />
 <!-- Laser and Link Laser-->
    <link name="laser">
     <inertial>
       <origin xyz="0 0 0" rpy="0 0 0" />
-      <mass value="1.2" />
-      <xacro:cylinder_inertia mass="1" r="0.05" l="0.1" />
+      <mass value="1.25" />
+      <xacro:cylinder_inertia mass="1.2" r="0.05" l="0.1" />
     </inertial>
     <visual>
@@ -116,10 +116,10 @@
   <link name="arm_base_link">
   	<inertial>
-  		<mass value="0.35"/>
-  		<origin xyz="0 0 0.085" rpy="0 1.57 0" />
+  		<mass value="0.27"/>
+  		<origin xyz="0 0 0.06" rpy="0 1.57 0" />
   		<inertia ixx="0.0000416666667" ixy="0" ixz="0" iyy="0.0000416666667" iyz="0" izz="0.0000416666667"/>
   	</inertial>
   	<collision>
-  	  <origin xyz="0 0 0.088" rpy="0 1.57 0"/>
+  	  <origin xyz="0 0 0.06" rpy="0 1.57 0"/>
       <geometry>
         <box size="0.12 0.12 0.47"/>
@@ -127,5 +127,5 @@
   	</collision>
   	<visual>
-  	  <origin xyz="0 0 0.085" rpy="0 1.57 0"/>
+  	  <origin xyz="0 0 0.06" rpy="0 1.57 0"/>
       <geometry>
         <box size="0.12 0.12 0.47"/>
@@ -142,5 +142,5 @@
   <link name="arm_link_01">
   	<inertial>
-  		<mass value="0.045"/>
+  		<mass value="0.025"/>
   		<origin xyz="0 0 0" rpy="0 0 0" />
   		<inertia ixx="0.000010279" ixy="0" ixz="0" iyy="0.000010279" iyz="0" izz="0.000007225"/>
@@ -149,5 +149,5 @@
   	  <origin xyz="0 0 0" rpy="0 0 0"/>
       <geometry>
-        <cylinder radius="0.045" length="0.36"/>
+        <cylinder radius="0.045" length="0.33"/>
       </geometry>
   	</collision>
@@ -155,5 +155,5 @@
   	  <origin xyz="0 0 0" rpy="0 0 0"/>
       <geometry>
-        <cylinder radius="0.045" length="0.36"/>
+        <cylinder radius="0.045" length="0.33"/>
       </geometry>
       <material name="red" />
@@ -162,6 +162,6 @@
   <joint name="arm_joint_01" type="revolute">
   	<axis xyz="0 0 1"/>
-  	<limit effort="1000.0" lower="-6.28" upper="6.28" velocity="0.55"/>
-  	<origin rpy="0 1.57 0" xyz="0.28 0 0.1"/>
+  	<limit effort="1000.0" lower="-6.28" upper="6.28" velocity="1"/>
+  	<origin rpy="0 1.57 0" xyz="0.18 0 0.05"/>
   	<parent link="arm_base_link"/>
   	<child link="arm_link_01"/>
@@ -169,5 +169,5 @@
     <link name="arm_link_02">
   	<inertial>
-  		<mass value="0.025"/>
+  		<mass value="0.015"/>
   		<origin xyz="0 0 0" rpy="0 0 0" />
   		<inertia ixx="0.000010279" ixy="0" ixz="0" iyy="0.000010279" iyz="0" izz="0.000007225"/>
@@ -176,5 +176,5 @@
   	  <origin xyz="0 0 0" rpy="0 0 0"/>
       <geometry>
-        <cylinder radius="0.04" length="0.5"/>
+        <cylinder radius="0.04" length="0.2"/>
       </geometry>
   	</collision>
@@ -182,5 +182,5 @@
   	  <origin xyz="0 0 0" rpy="0 0 0"/>
       <geometry>
-        <cylinder radius="0.04" length="0.5"/>
+        <cylinder radius="0.04" length="0.2"/>
       </geometry>
       <material name="red" />
@@ -189,6 +189,6 @@
   <joint name="arm_joint_02" type="revolute">
   	<axis xyz="0 0 1"/>
-  	<limit effort="1000.0" lower="-6.28" upper="6.28" velocity="0.4"/>
-  	<origin rpy="2 0 0" xyz="0 0.17 0.3"/>
+  	<limit effort="1000.0" lower="-6.28" upper="6.28" velocity="0.8"/>
+  	<origin rpy="2 0 0" xyz="0 0.08 0.2"/>
   	<parent link="arm_link_01"/>
   	<child link="arm_link_02"/>
@@ -196,18 +196,18 @@
       <link name="arm_link_03">
   	<inertial>
-  		<mass value="0.008"/>
-  		<origin xyz="0 0 0.32" rpy="0 0 0" />
-  		<inertia ixx="0.000010279" ixy="0" ixz="0" iyy="0.000010279" iyz="0" izz="0.000007225"/>
-  	</inertial>
-  	<collision>
-  	  <origin xyz="0 0 0.32" rpy="0 0 0"/>
-      <geometry>
-        <cylinder radius="0.035" length="0.55"/>
-      </geometry>
-  	</collision>
-  	<visual>
-  	  <origin xyz="0 0 0.32" rpy="0 0 0"/>
-      <geometry>
-        <cylinder radius="0.035" length="0.55"/>
+  		<mass value="0.004"/>
+  		<origin xyz="0 0 0.15" rpy="0 0 0" />
+  		<inertia ixx="0.000010279" ixy="0" ixz="0" iyy="0.000010279" iyz="0" izz="0.000007225"/>
+  	</inertial>
+  	<collision>
+  	  <origin xyz="0 0 0.15" rpy="0 0 0"/>
+      <geometry>
+        <cylinder radius="0.035" length="0.35"/>
+      </geometry>
+  	</collision>
+  	<visual>
+  	  <origin xyz="0 0 0.15" rpy="0 0 0"/>
+      <geometry>
+        <cylinder radius="0.035" length="0.35"/>
       </geometry>
       <material name="red" />
@@ -216,6 +216,6 @@
   <joint name="arm_joint_03" type="revolute">
   	<axis xyz="0 0 1"/>
-  	<limit effort="1000.0" lower="-6.28" upper="6.28" velocity="0.4"/>
-  	<origin rpy="-1.57 0 0" xyz="0 0 -0.22"/>
+  	<limit effort="1000.0" lower="-6.28" upper="6.28" velocity="0.6"/>
+  	<origin rpy="-1.57 0 0" xyz="0 0 -0.12"/>
   	<parent link="arm_link_02"/>
   	<child link="arm_link_03"/>
@@ -223,5 +223,5 @@
     <link name="arm_link_04">
   	<inertial>
-  		<mass value="0.007"/>
+  		<mass value="0.002"/>
   		<origin xyz="0 0 0.047" rpy="0 0 0" />
   		<inertia ixx="0.000010279" ixy="0" ixz="0" iyy="0.000010279" iyz="0" izz="0.000007225"/>
@@ -243,6 +243,6 @@
   <joint name="arm_joint_04" type="revolute">
   	<axis xyz="1 0 0"/>
-  	<limit effort="1000.0" lower="-6.28" upper="6.28" velocity="0.77"/>
-  	<origin rpy="0 0 0" xyz="0 0 0.58"/>
+  	<limit effort="1000.0" lower="-6.28" upper="6.28" velocity="0.5"/>
+  	<origin rpy="0 0 0" xyz="0 0 0.31"/>
   	<parent link="arm_link_03"/>
   	<child link="arm_link_04"/>
@@ -250,5 +250,5 @@
 <link name="cluedo_link">
   	<inertial>
-  		<mass value="0.007"/>
+  		<mass value="0.002"/>
   		<origin xyz="0 0 0" rpy="0 0 0" />
   		<inertia ixx="0.000010279" ixy="0" ixz="0" iyy="0.000010279" iyz="0" izz="0.000007225"/>
@@ -270,5 +270,5 @@
   <joint name="cluedo_joint" type="prismatic">
   	<axis xyz="1 0 0"/>
-  	<limit effort="1000.0" lower="-0.04" upper="0.035" velocity="6.6"/>
+  	<limit effort="1000.0" lower="-0.04" upper="0.035" velocity="1"/>
   	<origin rpy="0 0 0" xyz="0 0 0"/>
   	<parent link="arm_link_04"/>

File: urdf/robot6.urdf (robot description, URDF)
Before this commit: robot m2wr, 11 links, 10 joints
Links:
- link arm_base_link: mass 0.35 -> 0.27
- link arm_link_01: mass 0.045 -> 0.025; geometry collision cylinder length=0.33 radius=0.045; visual cylinder length=0.33 radius=0.045
- link arm_link_02: mass 0.025 -> 0.015; geometry collision cylinder length=0.2 radius=0.04; visual cylinder length=0.2 radius=0.04
- link arm_link_03: mass 0.008 -> 0.004; geometry collision cylinder length=0.35 radius=0.035; visual cylinder length=0.35 radius=0.035
- link arm_link_04: mass 0.007 -> 0.002
- link base_link: mass 10 -> 12; geometry collision box size=0.5 0.4 0.07; collision sphere radius=0.05
- link cluedo_link: mass 0.007 -> 0.002
- link laser: mass 1.2 -> 1.25
- link link_left_wheel: mass 0.2 -> 0.8
- link link_right_wheel: mass 0.2 -> 0.8
Joints:
- joint arm_joint_01: limit lower=-6.28 upper=6.28 effort=1000.0 velocity=0.55 -> lower=-6.28 upper=6.28 effort=1000.0 velocity=1; origin xyz=0.28 0 0.1 rpy=0 1.57 0 -> xyz=0.18 0 0.05 rpy=0 1.57 0
- joint arm_joint_02: limit lower=-6.28 upper=6.28 effort=1000.0 velocity=0.4 -> lower=-6.28 upper=6.28 effort=1000.0 velocity=0.8; origin xyz=0 0.17 0.3 rpy=2 0 0 -> xyz=0 0.08 0.2 rpy=2 0 0
- joint arm_joint_03: limit lower=-6.28 upper=6.28 effort=1000.0 velocity=0.4 -> lower=-6.28 upper=6.28 effort=1000.0 velocity=0.6; origin xyz=0 0 -0.22 rpy=-1.57 0 0 -> xyz=0 0 -0.12 rpy=-1.57 0 0
- joint arm_joint_04: limit lower=-6.28 upper=6.28 effort=1000.0 velocity=0.77 -> lower=-6.28 upper=6.28 effort=1000.0 velocity=0.5; origin xyz=0 0 0.58 rpy=0 0 0 -> xyz=0 0 0.31 rpy=0 0 0
- joint cluedo_joint: limit lower=-0.04 upper=0.035 effort=1000.0 velocity=6.6 -> lower=-0.04 upper=0.035 effort=1000.0 velocity=1
- joint joint_left_wheel: origin xyz=-0.05 0.15 0 rpy=0 0 0 -> xyz=-0.05 0.22 0 rpy=0 0 0
- joint joint_right_wheel: origin xyz=-0.05 -0.15 0 rpy=0 0 0 -> xyz=-0.05 -0.22 0 rpy=0 0 0

Commit message: TO DO: debug investigation, go to oracle and assert. Then write docs and README

File: urdf/m2wr_arm.xacro (robot description, xacro)
@@ -135,5 +135,5 @@
   </link>
   <joint name="arm_base_to_base" type="prismatic">
-    <limit effort="1000.0" lower="0" upper="0.32" velocity="1.5"/>
+    <limit effort="1000.0" lower="0" upper="0.32" velocity="0.2"/>
   	<origin rpy="0 -1.57 0" xyz="0 0 0.17"/>
   	<parent link="base_link"/>
@@ -162,5 +162,5 @@
   <joint name="arm_joint_01" type="revolute">
   	<axis xyz="0 0 1"/>
-  	<limit effort="1000.0" lower="-6.28" upper="6.28" velocity="1"/>
+  	<limit effort="1000.0" lower="-6.28" upper="6.28" velocity="0.2"/>
   	<origin rpy="0 1.57 0" xyz="0.18 0 0.05"/>
   	<parent link="arm_base_link"/>
@@ -189,5 +189,5 @@
   <joint name="arm_joint_02" type="revolute">
   	<axis xyz="0 0 1"/>
-  	<limit effort="1000.0" lower="-6.28" upper="6.28" velocity="0.8"/>
+  	<limit effort="1000.0" lower="-6.28" upper="6.28" velocity="0.2"/>
   	<origin rpy="2 0 0" xyz="0 0.08 0.2"/>
   	<parent link="arm_link_01"/>
@@ -216,5 +216,5 @@
   <joint name="arm_joint_03" type="revolute">
   	<axis xyz="0 0 1"/>
-  	<limit effort="1000.0" lower="-6.28" upper="6.28" velocity="0.6"/>
+  	<limit effort="1000.0" lower="-6.28" upper="6.28" velocity="0.2"/>
   	<origin rpy="-1.57 0 0" xyz="0 0 -0.12"/>
   	<parent link="arm_link_02"/>
@@ -243,5 +243,5 @@
   <joint name="arm_joint_04" type="revolute">
   	<axis xyz="1 0 0"/>
-  	<limit effort="1000.0" lower="-6.28" upper="6.28" velocity="0.5"/>
+  	<limit effort="1000.0" lower="-6.28" upper="6.28" velocity="0.4"/>
   	<origin rpy="0 0 0" xyz="0 0 0.31"/>
   	<parent link="arm_link_03"/>
@@ -270,5 +270,5 @@
   <joint name="cluedo_joint" type="prismatic">
   	<axis xyz="1 0 0"/>
-  	<limit effort="1000.0" lower="-0.04" upper="0.035" velocity="1"/>
+  	<limit effort="1000.0" lower="-0.04" upper="0.035" velocity="0.1"/>
   	<origin rpy="0 0 0" xyz="0 0 0"/>
   	<parent link="arm_link_04"/>

File: urdf/robot6.urdf (robot description, URDF)
Before this commit: robot m2wr, 11 links, 10 joints
Joints:
- joint arm_base_to_base: limit lower=0 upper=0.32 effort=1000.0 velocity=1.5 -> lower=0 upper=0.32 effort=1000.0 velocity=0.2
- joint arm_joint_01: limit lower=-6.28 upper=6.28 effort=1000.0 velocity=1 -> lower=-6.28 upper=6.28 effort=1000.0 velocity=0.2
- joint arm_joint_02: limit lower=-6.28 upper=6.28 effort=1000.0 velocity=0.8 -> lower=-6.28 upper=6.28 effort=1000.0 velocity=0.2
- joint arm_joint_03: limit lower=-6.28 upper=6.28 effort=1000.0 velocity=0.6 -> lower=-6.28 upper=6.28 effort=1000.0 velocity=0.2
- joint arm_joint_04: limit lower=-6.28 upper=6.28 effort=1000.0 velocity=0.5 -> lower=-6.28 upper=6.28 effort=1000.0 velocity=0.4
- joint cluedo_joint: limit lower=-0.04 upper=0.035 effort=1000.0 velocity=1 -> lower=-0.04 upper=0.035 effort=1000.0 velocity=0.1
